File: adapter/adapter.kicad_sch (KiCad schematic)
At the start: 13 parts, among them J1 AudioJack4, J2 AudioJack4, J3 Conn_01x02_Female, J4 Conn_01x03_Female, J5 Conn_01x03_Female, J6 Conn_01x02_Female, J7 Conn_01x06_Female, J9 Conn_01x06_Female, SW1 SW_SPST, SW2 SW_SPST, U1 eliteC, U2 eliteC, U3 YAAJ_WeAct_BlackPill_Part_Lik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

Commit message: pinout
Parts:
- removed U3: YAAJ_WeAct_BlackPill_Part_Like_SWD_Breakout, Library:YAAJ_WeAct_BlackPill_SWD_2, symbol YAAJ_WeAct_BlackPill_Part_Like_SWD_Breakout:YAAJ_WeAct_BlackPill_Part_Like_SWD_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
- added J?: AudioJack4, Library:Jack_3.5mm_PJ320E_Horizontal, symbol Connector:AudioJack4
- added R?: R, symbol Device:R
- added U?: YAAJ_WeAct_BlackPill_Part_Like_SWD_Breakout, Library:YAAJ_WeAct_BlackPill_SWD_2, symbol YAAJ_WeAct_BlackPill_Part_Like_SWD_Breakout:YAAJ_WeAct_BlackPill_Part_Like_SWD_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
Connections:
- net Din: no longer J4.3 (Pin_3)
- net Vcc: now also J?.T, R?.1, U?.18 (5V), U?.40 (5V)
- net Gnd renamed +5V
- net +5V: now also J?.R1, U?.19 (GND), U?.39 (GND)
- new net RGB_Din: J4.3 (Pin_3), R?.2, U?.27 (PA1)
- new net col1: U?.4 (PB15)
- new net col2: U?.3 (PB14)
- new net col3: U?.1 (PB12)
- new net col4: U?.14 (PB6)
- new net col5: U?.15 (PB7)
- new net col6: U?.16 (PB8)
- new net row1: U?.2 (PB13)
- new net row2: U?.6 (PA9)
- new net row3: U?.13 (PB5)
- new net row4: U?.12 (PB4)
- new net row5: U?.17 (PB9)
- new net serial: J?.R2, U?.10 (PA15)
- no-connect marks 34 -> 39
Other:
- note added: "RGB"
- note added: "Serial"
- note added: "Trackball connection"
- moved on the sheet: J4, J5, J7

Commit message: wiring
Parts:
- added R? (x2): 10k, symbol Device:R
- R?: value R -> 5.1k
Connections:
- net +5V: now also R?.2
- net Vcc: now also R?.1
- net miso: now also U?.32 (PA6)
- net mosi: now also U?.33 (PA7)
- net sc: now also U?.31 (PA5)
- net ss: now also U?.34 (PB0)
- net split_hand: now reaches U?.22 (PC13)
- net split_hand: now also R?.1
- net at U?.7 (PA10): now also R?.2
- no-connect marks 39 -> 38
Other:
- moved on the sheet: R?
Changed lines of the file:
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@@
 (kicad_sch (version 20210126) (generator eeschema)
   (paper "A4")
-  (junction (at 228.6 125.73) (diameter 1.016) (color 0 0 0 0))
   (no_connect (at 71.12 69.215))
   (no_connect (at 71.12 130.175))
@@
   (no_connect (at 123.19 143.51))
   (no_connect (at 123.19 153.67))
-  (no_connect (at 176.276 107.95))
   (no_connect (at 221.996 118.11))
   (no_connect (at 221.996 120.65))
@@
     (stroke (width 0) (type solid) (color 0 0 0 0))
   )
-  (wire (pts (xy 221.996 125.73) (xy 228.6 125.73))
-    (stroke (width 0) (type solid) (color 0 0 0 0))
-  )
-  (wire (pts (xy 228.6 125.73) (xy 228.6 122.682))
-    (stroke (width 0) (type solid) (color 0 0 0 0))
-  )
-  (wire (pts (xy 231.902 125.73) (xy 228.6 125.73))
+  (wire (pts (xy 158.75 94.996) (xy 158.75 99.314))
+    (stroke (width 0) (type solid) (color 0 0 0 0))
+  )
+  (wire (pts (xy 158.75 107.95) (xy 158.75 106.934))
+    (stroke (width 0) (type solid) (color 0 0 0 0))
+  )
+  (wire (pts (xy 176.276 107.95) (xy 158.75 107.95))
+    (stroke (width 0) (type solid) (color 0 0 0 0))
+  )
+  (wire (pts (xy 210.058 157.988) (xy 210.058 161.29))
+    (stroke (width 0) (type solid) (color 0 0 0 0))
+  )
+  (wire (pts (xy 228.346 159.004) (xy 233.172 159.004))
+    (stroke (width 0) (type solid) (color 0 0 0 0))
+  )
+  (wire (pts (xy 228.346 161.036) (xy 228.346 159.004))
+    (stroke (width 0) (type solid) (color 0 0 0 0))
+  )
+  (wire (pts (xy 228.346 168.656) (xy 228.346 172.72))
     (stroke (width 0) (type solid) (color 0 0 0 0))
   )
@@
     )
   )
+  (global_label "Vcc" (shape input) (at 158.75 94.996 90)
+    (effects (font (size 1.27 1.27)) (justify left))
+    (property "Intersheet References" "${INTERSHEET_REFS}" (id 0) (at 230.505 -49.149 0)
+      (effects (font (size 1.27 1.27)) hide)
+    )
+  )
   (global_label "col3" (shape input) (at 176.276 92.71 180)
     (effects (font (size 1.27 1.27)) (justify right))
@@
     )
   )
+  (global_label "Vcc" (shape input) (at 210.058 150.368 90)
+    (effects (font (size 1.27 1.27)) (justify left))
+    (property "Intersheet References" "${INTERSHEET_REFS}" (id 0) (at 281.813 6.223 0)
+      (effects (font (size 1.27 1.27)) hide)
+    )
+  )
+  (global_label "RGB_Din" (shape input) (at 210.058 161.29 0)
+    (effects (font (size 1.27 1.27)) (justify left))
+    (property "Intersheet References" "${INTERSHEET_REFS}" (id 0) (at 220.2725 161.2106 0)
+      (effects (font (size 1.27 1.27)) (justify left) hide)
+    )
+  )
   (global_label "Vcc" (shape input) (at 221.996 92.71 0)
     (effects (font (size 1.27 1.27)) (justify left))
@@
     )
   )
-  (global_label "Vcc" (shape input) (at 228.6 115.062 90)
-    (effects (font (size 1.27 1.27)) (justify left))
-    (property "Intersheet References" "${INTERSHEET_REFS}" (id 0) (at 300.355 -29.083 0)
-      (effects (font (size 1.27 1.27)) hide)
-    )
-  )
-  (global_label "RGB_Din" (shape input) (at 231.902 125.73 0)
-    (effects (font (size 1.27 1.27)) (justify left))
-    (property "Intersheet References" "${INTERSHEET_REFS}" (id 0) (at 242.1165 125.6506 0)
+  (global_label "ss" (shape input) (at 221.996 107.95 0)
+    (effects (font (size 1.27 1.27)) (justify left))
+    (property "Intersheet References" "${INTERSHEET_REFS}" (id 0) (at 226.4653 108.0294 0)
+      (effects (font (size 1.27 1.27)) (justify left) hide)
+    )
+  )
+  (global_label "mosi" (shape input) (at 221.996 110.49 0)
+    (effects (font (size 1.27 1.27)) (justify left))
+    (property "Intersheet References" "${INTERSHEET_REFS}" (id 0) (at 228.8843 110.5694 0)
+      (effects (font (size 1.27 1.27)) (justify left) hide)
+    )
+  )
+  (global_label "miso" (shape input) (at 221.996 113.03 0)
+    (effects (font (size 1.27 1.27)) (justify left))
+    (property "Intersheet References" "${INTERSHEET_REFS}" (id 0) (at 228.8843 113.1094 0)
+      (effects (font (size 1.27 1.27)) (justify left) hide)
+    )
+  )
+  (global_label "sc" (shape input) (at 221.996 115.57 0)
+    (effects (font (size 1.27 1.27)) (justify left))
+    (property "Intersheet References" "${INTERSHEET_REFS}" (id 0) (at 226.5258 115.6494 0)
+      (effects (font (size 1.27 1.27)) (justify left) hide)
+    )
+  )
+  (global_label "RGB_Din" (shape input) (at 221.996 125.73 0)
+    (effects (font (size 1.27 1.27)) (justify left))
+    (property "Intersheet References" "${INTERSHEET_REFS}" (id 0) (at 232.2105 125.6506 0)
+      (effects (font (size 1.27 1.27)) (justify left) hide)
+    )
+  )
+  (global_label "split_hand" (shape input) (at 221.996 138.43 0)
+    (effects (font (size 1.27 1.27)) (justify left))
+    (property "Intersheet References" "${INTERSHEET_REFS}" (id 0) (at 234.1458 138.3506 0)
+      (effects (font (size 1.27 1.27)) (justify left) hide)
+    )
+  )
+  (global_label "split_hand" (shape input) (at 233.172 159.004 0)
+    (effects (font (size 1.27 1.27)) (justify left))
+    (property "Intersheet References" "${INTERSHEET_REFS}" (id 0) (at 245.3218 158.9246 0)
       (effects (font (size 1.27 1.27)) (justify left) hide)
     )
@@
       (effects (font (size 1.27 1.27)) hide)
     )
+  )
+  (symbol (lib_id "keyboard_parts:GND") (at 228.346 172.72 0) (unit 1)
+    (in_bom yes) (on_board yes)
+    (property "Reference" "#PWR?" (id 0) (at 228.346 171.45 0)
+      (effects (font (size 0.508 0.508)) hide)
+    )
+    (property "Value" "GND" (id 1) (at 228.981 170.815 0)
+      (effects (font (size 0.762 0.762)))
+    )
+    (property "Footprint" "" (id 2) (at 228.346 172.72 0)
+      (effects (font (size 1.524 1.524)))
+    )
+    (property "Datasheet" "" (id 3) (at 228.346 172.72 0)
+      (effects (font (size 1.524 1.524)))
+    )
+    (pin "1")
   )
   (symbol (lib_id "keyboard_parts:GND") (at 262.255 132.08 0) (unit 1)
@@
     (pin "1")
   )
-  (symbol (lib_id "Device:R") (at 228.6 118.872 0) (unit 1)
-    (in_bom yes) (on_board yes)
-    (property "Reference" "R?" (id 0) (at 231.14 117.602 0)
-      (effects (font (size 1.27 1.27)) (justify left))
-    )
-    (property "Value" "R" (id 1) (at 231.14 120.142 0)
-      (effects (font (size 1.27 1.27)) (justify left))
-    )
-    (property "Footprint" "" (id 2) (at 226.822 118.872 90)
-      (effects (font (size 1.27 1.27)) hide)
-    )
-    (property "Datasheet" "~" (id 3) (at 228.6 118.872 0)
+  (symbol (lib_id "Device:R") (at 158.75 103.124 0) (unit 1)
+    (in_bom yes) (on_board yes)
+    (property "Reference" "R?" (id 0) (at 161.29 101.854 0)
+      (effects (font (size 1.27 1.27)) (justify left))
+    )
+    (property "Value" "10k" (id 1) (at 161.29 104.394 0)
+      (effects (font (size 1.27 1.27)) (justify left))
+    )
+    (property "Footprint" "" (id 2) (at 156.972 103.124 90)
+      (effects (font (size 1.27 1.27)) hide)
+    )
+    (property "Datasheet" "~" (id 3) (at 158.75 103.124 0)
+      (effects (font (size 1.27 1.27)) hide)
+    )
+    (pin "1")
+    (pin "2")
+  )
+  (symbol (lib_id "Device:R") (at 210.058 154.178 0) (unit 1)
+    (in_bom yes) (on_board yes)
+    (property "Reference" "R?" (id 0) (at 212.09 153.67 0)
+      (effects (font (size 1.27 1.27)) (justify left))
+    )
+    (property "Value" "5.1k" (id 1) (at 212.09 156.21 0)
+      (effects (font (size 1.27 1.27)) (justify left))
+    )
+    (property "Footprint" "" (id 2) (at 208.28 154.178 90)
+      (effects (font (size 1.27 1.27)) hide)
+    )
+    (property "Datasheet" "~" (id 3) (at 210.058 154.178 0)
+      (effects (font (size 1.27 1.27)) hide)
+    )
+    (pin "1")
+    (pin "2")
+  )
+  (symbol (lib_id "Device:R") (at 228.346 164.846 0) (unit 1)
+    (in_bom yes) (on_board yes)
+    (property "Reference" "R?" (id 0) (at 230.886 163.576 0)
+      (effects (font (size 1.27 1.27)) (justify left))
+    )
+    (property "Value" "10k" (id 1) (at 230.886 166.116 0)
+      (effects (font (size 1.27 1.27)) (justify left))
+    )
+    (property "Footprint" "" (id 2) (at 226.568 164.846 90)
+      (effects (font (size 1.27 1.27)) hide)
+    )
+    (property "Datasheet" "~" (id 3) (at 228.346 164.846 0)
       (effects (font (size 1.27 1.27)) hide)
     )
@@
   )
   (symbol_instances
+    (path "/314649fe-ba68-4398-8b6b-73118e638aeb"
+      (reference "#PWR?") (unit 1) (value "GND") (footprint "")
+    )
     (path "/d4134c27-23ab-4c53-ab29-85c12b0db249"
       (reference "#PWR?") (unit 1) (value "GND") (footprint "")
@@
       (reference "J?") (unit 1) (value "AudioJack4") (footprint "Library:Jack_3.5mm_PJ320E_Horizontal")
     )
+    (path "/31a6626f-f424-4420-98bb-68e70d330bba"
+      (reference "R?") (unit 1) (value "10k") (footprint "")
+    )
+    (path "/a9010c44-9f41-4444-bd4c-d23a0eb584a6"
+      (reference "R?") (unit 1) (value "10k") (footprint "")
+    )
     (path "/d6cbb0a1-7ce9-402e-b509-2198e9b3dfdc"
-      (reference "R?") (unit 1) (value "R") (footprint "")
+      (reference "R?") (unit 1) (value "5.1k") (footprint "")
     )
     (path "/0b28cd91-b5a2-4261-9655-460b63454a83"

Commit message: Small overhaul
Parts:
- added R?: 5.1k, symbol Device:R
- J4: value Conn_01x03_Female -> RGB
- J7: value Conn_01x06_Female -> Trackball
- J?: value AudioJack4 -> Serial
- R? (x2): value 10k -> 5.1k
- U?: value YAAJ_WeAct_BlackPill_Part_Like_SWD_Breakout -> STM32F401 / STM32F411 Blackpill Breakout
Connections:
- net Vcc: now also R?.1
- net row2: no longer U?.6 (PA9)
- net serial: now also R?.2; no longer U?.10 (PA15)
- net split_hand: now also R?.2, U?.23 (PC14), R?.1; no longer R?.1, U?.22 (PC13)
- net at U?.7 (PA10): no longer R?.2
- removed net +5V: J1.R1, J4.2 (Pin_2), J7.6 (Pin_6), J?.R1, R?.2, SW1.2 (B), U1.23 (GND), U1.3 (GND), U1.4 (GND), U?.19 (GND), U?.39 (GND)
- net RGB_Din renamed RGB
- net sc renamed sck
- net sc2 renamed sck2
- net ss renamed ss_trackball
- net ss_trackball: no longer U?.34 (PB0)
- net ss2 renamed ss_trackball2
- new net GND: J4.2 (Pin_2), J7.6 (Pin_6), J?.R1, R?.2, U?.19 (GND), U?.39 (GND)
- new net Gnd: J1.R1, SW1.2 (B), U1.23 (GND), U1.3 (GND), U1.4 (GND)
- no-connect marks 38 -> 44
Other:
- note added: "Blackpill Boards have a SOIC-8 footprint for SPI 25x EEPROMS on the backside. This EEPROM is wired up to the SPI1 peripheral, which is also connected to the trackball. To signal which device should use the SPI bus we use different Chip Select / SS pins. As the EEPROMs CS pin is already connected to PA4 we have to choose another pin."
- note added: "Connectors"
- note added: "Handedness selection works by removing one of the resistors, so that the pin is either pulled low or high. This is checked upon boot and the correct side is set at runtime."
- note added: "MCU"
- note added: "OG Blackpill Schematics are under the docs folder."
- note added: "Pull-ups / Pull-downs"
- note added: "Serial split comms in Half-duplex mode operate the TX pin in open drain configuration. Therefore a pull-up resistor is needed."
- note added: "The PWM driver for the WS2812 and SK6812 LEDs operate the PWM pin in open drain configuration. Therefore a pull-up resistor is needed."
- note removed: "RGB"
- note removed: "Serial"
- note removed: "Trackball connection"
- moved on the sheet: J1, J2, J3, J4, J5, J6, J7, J9, J?, R?, SW1, SW2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

Commit message: Add Datasheets / Refecrence manuals, correct 5V and 3.3V usage
Parts:
- added SW?: Reset, customs:switch_rst, symbol Switch:SW_SPST
Connections:
- net GND: now also SW?.2 (B)
- net Vcc: no longer J4.1 (Pin_1), J7.1 (Pin_1), J?.T, R?.1, R?.1, R?.1, U?.40 (5V)
- net split_hand: now also U?.26 (PA0); no longer U?.23 (PC14)
- net +3V3: now reaches U?.20 (3V3)
- net +3V3: now also R?.1, R?.1
- net NRST: now reaches U?.25 (RES)
- net NRST: now also SW?.1 (A)
- new net +5V: J4.1 (Pin_1), J7.1 (Pin_1), J?.T, R?.1, U?.40 (5V)
- no-connect marks 44 -> 46
Other:
- note added: "Switch"
- note added: "The PWM driver for the WS2812 and SK6812 LEDs operate the PWM pin in open drain configuration. Therefore a pull-up resistor to 5V is needed, as the LEDs use their supply voltage as signaling level."
- note removed: "The PWM driver for the WS2812 and SK6812 LEDs operate the PWM pin in open drain configuration. Therefore a pull-up resistor is needed."

Commit message: row and col connectors
Parts:
- removed J1, J2: AudioJack4, Library:Jack_3.5mm_PJ320E_Horizontal, symbol Connector:AudioJack4
- removed J3, J6: Conn_01x02_Female, Connector_PinSocket_2.54mm:PinSocket_2x01_P2.54mm_Vertical, symbol Connector:Conn_01x02_Female
- removed J5: Conn_01x03_Female, Connector_PinSocket_2.54mm:PinSocket_1x03_P2.54mm_Vertical, symbol Connector:Conn_01x03_Female
- removed J9: Conn_01x06_Female, Connector_PinHeader_2.54mm:PinHeader_1x06_P2.54mm_Vertical, symbol Connector:Conn_01x06_Female
- removed SW1, SW2: SW_SPST, customs:switch_rst, symbol Switch:SW_SPST
- removed U1, U2: eliteC, Library:Elite-C-castellated-29pin-holes, symbol elite-C:eliteC
- added J2: Conn_01x05_Female, customs:PinHeader_1x05_P2.54mm_Vertical, symbol Connector:Conn_01x05_Female
- added J3: Conn_01x06_Female, Connector_PinHeader_2.54mm:PinHeader_1x06_P2.54mm_Vertical, symbol Connector:Conn_01x06_Female
- gave numbers to parts that had none: 7
Connections:
- net col1: now also J2.4 (Pin_4)
- net col2: now also J2.3 (Pin_3)
- net col3: now also J2.1 (Pin_1)
- net col4: now also J3.3 (Pin_3)
- net col5: now also J3.4 (Pin_4)
- net col6: now also J3.5 (Pin_5)
- net row1: now also J2.2 (Pin_2)
- net row2: now also J2.5 (Pin_5)
- net row3: now also J3.2 (Pin_2)
- net row4: now also J3.1 (Pin_1)
- net row5: now also J3.6 (Pin_6)
- no-connect marks 46 -> 12
Other:
- note added: "Rows and Columns"
- moved on the sheet: J1, J4, J7, R1, R2, R3, R4, SW1, U1

Commit message: Update schematic for left and right hand
Parts:
- removed J2: Conn_01x05_Female, customs:PinHeader_1x05_P2.54mm_Vertical, symbol Connector:Conn_01x05_Female
- removed J3: Conn_01x06_Female, Connector_PinHeader_2.54mm:PinHeader_1x06_P2.54mm_Vertical, symbol Connector:Conn_01x06_Female
- removed SW1: Reset, customs:switch_rst, symbol Switch:SW_SPST
- added J2: Serial, Library:Jack_3.5mm_PJ320E_Horizontal, symbol Connector:AudioJack4
- added J3: RGB, Connector_PinSocket_2.54mm:PinSocket_1x03_P2.54mm_Vertical, symbol Connector:Conn_01x03_Female
- added J5: Trackball, Connector_PinHeader_2.54mm:PinHeader_1x06_P2.54mm_Vertical, symbol Connector:Conn_01x06_Female
- added J? (x2): Ribbon, customs:PinHeader_1x05_P2.54mm_Vertical, symbol Connector:Conn_01x05_Female
- added J? (x2): Ribbon, Connector_PinHeader_2.54mm:PinHeader_1x06_P2.54mm_Vertical, symbol Connector:Conn_01x06_Female
- added R1, R5, R6, R7: 5.1k, Resistor_SMD:R_0805_2012Metric_Pad1.20x1.40mm_HandSolder, symbol Device:R
- added U1: STM32F401 / STM32F411 Blackpill Breakout, Library:YAAJ_WeAct_BlackPill_SWD_2, symbol YAAJ_WeAct_BlackPill_Part_Like_SWD_Breakout:YAAJ_WeAct_BlackPill_Part_Like_SWD_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
- J1, J4, J7: JLCPCB BOM (none) -> 0
- R2: renamed from R1; footprint (none) -> Resistor_SMD:R_0805_2012Metric_Pad1.20x1.40mm_HandSolder; JLCPCB BOM (none) -> 1; JLCPCB Part (none) -> C27834
- R3, R4: footprint (none) -> Resistor_SMD:R_0805_2012Metric_Pad1.20x1.40mm_HandSolder; JLCPCB BOM (none) -> 1; JLCPCB Part (none) -> C27834
- R8: renamed from R2; footprint (none) -> Resistor_SMD:R_0805_2012Metric_Pad1.20x1.40mm_HandSolder; JLCPCB BOM (none) -> 1; JLCPCB Part (none) -> C27834
- U2: renamed from U1; JLCPCB BOM (none) -> 0
Connections:
- net Vcc is gone; now on net +5V: U2.18 (5V)
- net +3V3: now also R1.1, R6.1, R7.1, U1.20 (3V3)
- net +5V: now also J2.T, J3.1 (Pin_1), J5.1 (Pin_1), R5.1, U1.18 (5V), U1.40 (5V)
- net GND: now also J2.R1, J3.2 (Pin_2), J5.6 (Pin_6), U1.19 (GND), U1.39 (GND)
- net ss_trackball_l: now reaches U2.10 (PA15)
- net ss_trackball_l: now also J5.2 (Pin_2)
- net col4_l: now reaches U2.11 (PB3)
- net col4_l: now also J?.3 (Pin_3)
- net col1_l: now reaches U2.34 (PB0)
- net col1_l: now also J?.4 (Pin_4)
- net col2_l: now reaches U2.35 (PB1)
- net col2_l: now also J?.3 (Pin_3)
- net col3_l: now reaches U2.36 (PB2)
- net col3_l: now also J?.1 (Pin_1)
- net dfu_bootloader_bodge_l: now reaches U2.7 (PA10)
- net dfu_bootloader_bodge_l: now also R1.2
- net NRST: no longer names the net of U2.25 (RES)
- net RGB renamed rgb_l
- net rgb_l: now also J3.3 (Pin_3); no longer J4.3 (Pin_3)
- net col1 renamed row4_l
- net row4_l: now also J?.1 (Pin_1)
- net col2 renamed row3_l
- net row3_l: now also J?.2 (Pin_2)
- net col3 renamed row1_l
- net row1_l: now also J?.2 (Pin_2)
- net col4 renamed row5_l
- net row5_l: now also J?.6 (Pin_6)
- net col5: no longer names the net of U2.15 (PB7)
- net col6: no longer names the net of U2.16 (PB8)
- net miso renamed miso_l
- net miso_l: now also J5.5 (Pin_5); no longer J7.5 (Pin_5)
- net mosi renamed mosi_l
- net mosi_l: now also J5.3 (Pin_3); no longer J7.3 (Pin_3)
- net row1 renamed row2_l
- net row2_l: now also J?.5 (Pin_5)
- net row3 renamed col6_l
- net col6_l: now also J?.5 (Pin_5)
- net row4 renamed col5_l
- net col5_l: now also J?.4 (Pin_4)
- net row5: no longer names the net of U2.17 (PB9)
- net sck renamed sck_l
- net sck_l: now also J5.4 (Pin_4); no longer J7.4 (Pin_4)
- net serial renamed serial_l
- net serial_l: now also J2.R2; no longer J1.R2
- net split_hand renamed split_hand_l
- net split_hand_l: no longer R8.1
- net ss_trackball renamed ss_trackball_r
- net ss_trackball_r: now also U1.10 (PA15)
- new net col1_r: J?.4 (Pin_4), U1.34 (PB0)
- new net col2_r: J?.3 (Pin_3), U1.35 (PB1)
- new net col3_r: J?.1 (Pin_1), U1.36 (PB2)
- new net col4_r: J?.3 (Pin_3), U1.11 (PB3)
- new net col5_r: J?.4 (Pin_4), U1.12 (PB4)
- new net col6_r: J?.5 (Pin_5), U1.13 (PB5)
- new net dfu_bootloader_bodge_r: R7.2, U1.7 (PA10)
- new net miso_r: J7.5 (Pin_5), U1.32 (PA6)
- new net mosi_r: J7.3 (Pin_3), U1.33 (PA7)
- new net rgb_r: J4.3 (Pin_3), R5.2, U1.27 (PA1)
- new net row1_r: J?.2 (Pin_2), U1.1 (PB12)
- new net row2_r: J?.5 (Pin_5), U1.2 (PB13)
- new net row3_r: J?.2 (Pin_2), U1.3 (PB14)
- new net row4_r: J?.1 (Pin_1), U1.4 (PB15)
- new net row5_r: J?.6 (Pin_6), U1.5 (PA8)
- new net sck_r: J7.4 (Pin_4), U1.31 (PA5)
- new net serial_r: J1.R2, R6.2
- new net split_hand_r: R8.1, U1.26 (PA0)
- no-connect marks 12 -> 28
Other:
- note added: "Early revisions of the STM32F1 and apparently STM32F4 USB-DFU bootloader had problems with entering a stable state. A workaround is simply to pull the PA10 pin into a permanent high state."
- note added: "Handedness selection works by pulling a dedicated pin high or low this is checked upon boot and the correct side is set at runtime. The default is high for the left side and low for the right side, but this can be overwritten in firmware."
- note added: "MCU Left"
- note added: "MCU Right"
- note removed: "Handedness selection works by removing one of the resistors, so that the pin is either pulled low or high. This is checked upon boot and the correct side is set at runtime."
- note removed: "MCU"
- note removed: "Rows and Columns"
- note removed: "Switch"
- company: (none) -> Bastardkb x KarlK90
- title: (none) -> Charybdis Blackpill Holder
- moved on the sheet: J1, J4, J7, R2, R3, R4, R8, U2

Commit message: fix connection placement
Parts:
- gave numbers to parts that had none: 4
Other:
- note added: "Connectors Left"
- note added: "Connectors Right"
- note removed: "Connectors"
- moved on the sheet: J1, J10, J2, J3, J4, J5, J6, J7, J8, J9

Commit message: component placement
Parts:
- J6: footprint customs:PinHeader_1x05_P2.54mm_Vertical -> Connector_PinHeader_2.54mm:PinHeader_1x05_P2.54mm_Vertical
Changed lines of the file:
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@@
       (effects (font (size 1.27 1.27)) (justify left))
     )
-    (property "Footprint" "customs:PinHeader_1x05_P2.54mm_Vertical" (id 2) (at 231.775 149.733 0)
+    (property "Footprint" "Connector_PinHeader_2.54mm:PinHeader_1x05_P2.54mm_Vertical" (id 2) (at 231.775 149.733 0)
       (effects (font (size 1.27 1.27)) hide)
     )
@@
     )
     (path "/45f0799c-408b-4e0d-8bc6-8ee6ccaf8219"
-      (reference "J6") (unit 1) (value "Ribbon") (footprint "customs:PinHeader_1x05_P2.54mm_Vertical")
+      (reference "J6") (unit 1) (value "Ribbon") (footprint "Connector_PinHeader_2.54mm:PinHeader_1x05_P2.54mm_Vertical")
     )
     (path "/7bffcea9-b23e-4698-8571-09d538a5c739"
