File: adapter/adapter.kicad_sch (KiCad schematic)
At the start: 20 parts, among them J1 Serial, J10 Ribbon, J2 Serial, J3 RGB, J4 RGB, J5 Trackball, J6 Ribbon, J7 Trackball, J8 Ribbon, J9 Ribbon, U1 STM32F401 / STM32F411 Blackpi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, U2 STM32F401 / STM32F411 Blackpi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

Commit message: component placement
Parts:
- R1, R2, R3, R4, R5, R6, R7, R8: footprint Resistor_SMD:R_0805_2012Metric_Pad1.20x1.40mm_HandSolder -> Resistor_SMD:R_1206_3216Metric_Pad1.30x1.75mm_HandSolder
Changed lines of the file:
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@@
       (effects (font (size 1.27 1.27)) (justify left))
     )
-    (property "Footprint" "Resistor_SMD:R_0805_2012Metric_Pad1.20x1.40mm_HandSolder" (id 2) (at 22.352 38.1 90)
+    (property "Footprint" "Resistor_SMD:R_1206_3216Metric_Pad1.30x1.75mm_HandSolder" (id 2) (at 22.352 38.1 90)
       (effects (font (size 1.27 1.27)) hide)
     )
@@
       (effects (font (size 1.27 1.27)) (justify left))
     )
-    (property "Footprint" "Resistor_SMD:R_0805_2012Metric_Pad1.20x1.40mm_HandSolder" (id 2) (at 32.512 141.605 90)
+    (property "Footprint" "Resistor_SMD:R_1206_3216Metric_Pad1.30x1.75mm_HandSolder" (id 2) (at 32.512 141.605 90)
       (effects (font (size 1.27 1.27)) hide)
     )
@@
       (effects (font (size 1.27 1.27)) (justify left))
     )
-    (property "Footprint" "Resistor_SMD:R_0805_2012Metric_Pad1.20x1.40mm_HandSolder" (id 2) (at 22.352 113.665 90)
+    (property "Footprint" "Resistor_SMD:R_1206_3216Metric_Pad1.30x1.75mm_HandSolder" (id 2) (at 22.352 113.665 90)
       (effects (font (size 1.27 1.27)) hide)
     )
@@
       (effects (font (size 1.27 1.27)) (justify left))
     )
-    (property "Footprint" "Resistor_SMD:R_0805_2012Metric_Pad1.20x1.40mm_HandSolder" (id 2) (at 35.052 37.465 90)
+    (property "Footprint" "Resistor_SMD:R_1206_3216Metric_Pad1.30x1.75mm_HandSolder" (id 2) (at 35.052 37.465 90)
       (effects (font (size 1.27 1.27)) hide)
     )
@@
       (effects (font (size 1.27 1.27)) (justify left))
     )
-    (property "Footprint" "Resistor_SMD:R_0805_2012Metric_Pad1.20x1.40mm_HandSolder" (id 2) (at 33.782 113.665 90)
+    (property "Footprint" "Resistor_SMD:R_1206_3216Metric_Pad1.30x1.75mm_HandSolder" (id 2) (at 33.782 113.665 90)
       (effects (font (size 1.27 1.27)) hide)
     )
@@
       (effects (font (size 1.27 1.27)) (justify left))
     )
-    (property "Footprint" "Resistor_SMD:R_0805_2012Metric_Pad1.20x1.40mm_HandSolder" (id 2) (at 22.352 78.74 90)
+    (property "Footprint" "Resistor_SMD:R_1206_3216Metric_Pad1.30x1.75mm_HandSolder" (id 2) (at 22.352 78.74 90)
       (effects (font (size 1.27 1.27)) hide)
     )
@@
       (effects (font (size 1.27 1.27)) (justify left))
     )
-    (property "Footprint" "Resistor_SMD:R_0805_2012Metric_Pad1.20x1.40mm_HandSolder" (id 2) (at 22.352 141.605 90)
+    (property "Footprint" "Resistor_SMD:R_1206_3216Metric_Pad1.30x1.75mm_HandSolder" (id 2) (at 22.352 141.605 90)
       (effects (font (size 1.27 1.27)) hide)
     )
@@
       (effects (font (size 1.27 1.27)) (justify left))
     )
-    (property "Footprint" "Resistor_SMD:R_0805_2012Metric_Pad1.20x1.40mm_HandSolder" (id 2) (at 35.052 90.805 90)
+    (property "Footprint" "Resistor_SMD:R_1206_3216Metric_Pad1.30x1.75mm_HandSolder" (id 2) (at 35.052 90.805 90)
       (effects (font (size 1.27 1.27)) hide)
     )
@@
     )
     (path "/2359a6b2-1ec9-424d-a02c-d839b6fe2dff"
-      (reference "R1") (unit 1) (value "5.1k") (footprint "Resistor_SMD:R_0805_2012Metric_Pad1.20x1.40mm_HandSolder")
+      (reference "R1") (unit 1) (value "5.1k") (footprint "Resistor_SMD:R_1206_3216Metric_Pad1.30x1.75mm_HandSolder")
     )
     (path "/a9010c44-9f41-4444-bd4c-d23a0eb584a6"
-      (reference "R2") (unit 1) (value "5.1k") (footprint "Resistor_SMD:R_0805_2012Metric_Pad1.20x1.40mm_HandSolder")
+      (reference "R2") (unit 1) (value "5.1k") (footprint "Resistor_SMD:R_1206_3216Metric_Pad1.30x1.75mm_HandSolder")
     )
     (path "/31a6626f-f424-4420-98bb-68e70d330bba"
-      (reference "R3") (unit 1) (value "5.1k") (footprint "Resistor_SMD:R_0805_2012Metric_Pad1.20x1.40mm_HandSolder")
+      (reference "R3") (unit 1) (value "5.1k") (footprint "Resistor_SMD:R_1206_3216Metric_Pad1.30x1.75mm_HandSolder")
     )
     (path "/d6cbb0a1-7ce9-402e-b509-2198e9b3dfdc"
-      (reference "R4") (unit 1) (value "5.1k") (footprint "Resistor_SMD:R_0805_2012Metric_Pad1.20x1.40mm_HandSolder")
+      (reference "R4") (unit 1) (value "5.1k") (footprint "Resistor_SMD:R_1206_3216Metric_Pad1.30x1.75mm_HandSolder")
     )
     (path "/31692d3a-9ca8-4b5c-9af3-2fdf59035dd6"
-      (reference "R5") (unit 1) (value "5.1k") (footprint "Resistor_SMD:R_0805_2012Metric_Pad1.20x1.40mm_HandSolder")
+      (reference "R5") (unit 1) (value "5.1k") (footprint "Resistor_SMD:R_1206_3216Metric_Pad1.30x1.75mm_HandSolder")
     )
     (path "/89a17716-30dd-4858-9688-3a8fdd26ea18"
-      (reference "R6") (unit 1) (value "5.1k") (footprint "Resistor_SMD:R_0805_2012Metric_Pad1.20x1.40mm_HandSolder")
+      (reference "R6") (unit 1) (value "5.1k") (footprint "Resistor_SMD:R_1206_3216Metric_Pad1.30x1.75mm_HandSolder")
     )
     (path "/69455eac-7ea1-4fa5-9c1f-8072a7c2bb2a"
-      (reference "R7") (unit 1) (value "5.1k") (footprint "Resistor_SMD:R_0805_2012Metric_Pad1.20x1.40mm_HandSolder")
+      (reference "R7") (unit 1) (value "5.1k") (footprint "Resistor_SMD:R_1206_3216Metric_Pad1.30x1.75mm_HandSolder")
     )
     (path "/f7a8ef2f-3545-4d15-89ff-8d21b81bb891"
-      (reference "R8") (unit 1) (value "5.1k") (footprint "Resistor_SMD:R_0805_2012Metric_Pad1.20x1.40mm_HandSolder")
+      (reference "R8") (unit 1) (value "5.1k") (footprint "Resistor_SMD:R_1206_3216Metric_Pad1.30x1.75mm_HandSolder")
     )
     (path "/38ec90f9-e990-409a-bb98-dd9a134e92d3"

Commit message: placement
Connections:
- net +5V: no longer U2.40 (5V)
- no-connect marks 28 -> 29
Changed lines of the file:
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@@
   (no_connect (at 137.795 168.275))
   (no_connect (at 205.994 35.941))
+  (no_connect (at 163.83 35.052))
   (no_connect (at 163.83 62.865))
   (no_connect (at 163.83 65.405))
@@
     (pin "1")
   )
-  (symbol (lib_id "power:+5V") (at 163.83 34.925 270) (unit 1)
-    (in_bom yes) (on_board yes) (fields_autoplaced)
-    (property "Reference" "#PWR0101" (id 0) (at 160.02 34.925 0)
-      (effects (font (size 1.27 1.27)) hide)
-    )
-    (property "Value" "+5V" (id 1) (at 167.005 35.404 90)
-      (effects (font (size 1.27 1.27)) (justify left))
-    )
-    (property "Footprint" "" (id 2) (at 163.83 34.925 0)
-      (effects (font (size 1.27 1.27)) hide)
-    )
-    (property "Datasheet" "" (id 3) (at 163.83 34.925 0)
-      (effects (font (size 1.27 1.27)) hide)
-    )
-    (pin "1")
-  )
   (symbol (lib_id "power:+3.3V") (at 36.83 33.655 0) (unit 1)
     (in_bom yes) (on_board yes) (fields_autoplaced)
@@
   )
   (symbol_instances
-    (path "/c302c14f-0f07-4722-9635-4326a484712c"
-      (reference "#PWR0101") (unit 1) (value "+5V") (footprint "")
-    )
     (path "/cf564857-3c48-44d0-a2b1-960c8d42cb17"
       (reference "#PWR0102") (unit 1) (value "GND") (footprint "")

Commit message: right edge cuts
Parts:
- J9: footprint customs:PinHeader_1x05_P2.54mm_Vertical -> Connector_PinHeader_2.54mm:PinHeader_1x05_P2.54mm_Vertical
Changed lines of the file:
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@@
       (effects (font (size 1.27 1.27)) (justify left))
     )
-    (property "Footprint" "customs:PinHeader_1x05_P2.54mm_Vertical" (id 2) (at 233.299 67.691 0)
+    (property "Footprint" "Connector_PinHeader_2.54mm:PinHeader_1x05_P2.54mm_Vertical" (id 2) (at 233.299 67.691 0)
       (effects (font (size 1.27 1.27)) hide)
     )
@@
     )
     (path "/fcc4bfec-a658-4f05-a805-e2fbe77edcaf"
-      (reference "J9") (unit 1) (value "Ribbon") (footprint "customs:PinHeader_1x05_P2.54mm_Vertical")
+      (reference "J9") (unit 1) (value "Ribbon") (footprint "Connector_PinHeader_2.54mm:PinHeader_1x05_P2.54mm_Vertical")
     )
     (path "/72f9f857-8d29-4f7f-9028-4223dc06e9cc"

Commit message: Traces for left side
Parts:
- added H1, H2, H3, H4: M4, Library:MountingHole_4mm_Pad_Thin, symbol Mechanical:MountingHole_Pad
- added J11, J12: SPI user, Library:6_PinHeader, symbol Connector:Conn_01x06_Female
- added SW1, SW2: USER, Library:PushSwitch, symbol Switch:SW_Push
- J10, J5, J7, J8: footprint Connector_PinHeader_2.54mm:PinHeader_1x06_P2.54mm_Vertical -> Library:6_PinHeader
- J3, J4: footprint Connector_PinSocket_2.54mm:PinSocket_1x03_P2.54mm_Vertical -> Library:3_PinSocket
- J6, J9: footprint Connector_PinHeader_2.54mm:PinHeader_1x05_P2.54mm_Vertical -> Library:5_PinHeader
- R1, R2, R3, R4, R5, R6, R7, R8: JLCPCB Part C27834 -> C26033
- U1, U2: footprint Library:YAAJ_WeAct_BlackPill_SWD_2 -> Library:WeAct_BlackPill_without_SWD_First_Row
Connections:
- net +3V3: now also U1.38 (3V3), U2.38 (3V3); no longer U1.20 (3V3), U2.20 (3V3)
- net +5V: now also J11.1 (Pin_1), J12.1 (Pin_1); no longer U1.40 (5V)
- net GND: now also H1.1, H2.1, H3.1, H4.1, J11.6 (Pin_6), J12.6 (Pin_6), SW1.2, SW2.2
- net miso_l: now also J11.5 (Pin_5)
- net miso_r: now also J12.5 (Pin_5)
- net mosi_l: now also J11.3 (Pin_3)
- net mosi_r: now also J12.3 (Pin_3)
- net row1_l: now also U2.4 (PB15); no longer U2.1 (PB12)
- net row1_r: now also U1.4 (PB15); no longer U1.1 (PB12)
- net row2_l: now also U2.28 (PA2); no longer U2.2 (PB13)
- net row2_r: now also U1.28 (PA2); no longer U1.2 (PB13)
- net row3_l: now also U2.16 (PB8); no longer U2.3 (PB14)
- net row3_r: now also U1.16 (PB8); no longer U1.3 (PB14)
- net row4_l: now also U2.5 (PA8); no longer U2.4 (PB15)
- net row4_r: now also U1.5 (PA8); no longer U1.4 (PB15)
- net row5_l: now also U2.17 (PB9); no longer U2.14 (PB6)
- net row5_r: now also U1.17 (PB9); no longer U1.5 (PA8)
- net sck_l: now also J11.4 (Pin_4)
- net sck_r: now also J12.4 (Pin_4)
- net serial_l: now also U2.6 (PA9)
- net split_hand_l: now also U2.29 (PA3); no longer U2.26 (PA0)
- net split_hand_r: now also U1.29 (PA3); no longer U1.26 (PA0)
- net scl_r: now reaches U1.14 (PB6)
- net sda_r: now reaches U1.15 (PB7)
- net sda_l: now reaches U2.15 (PB7)
- net ss_trackball_l renamed cs_trackball_l
- net cs_trackball_l: now also U2.3 (PB14); no longer U2.10 (PA15)
- net ss_trackball_r renamed cs_trackball_r
- net cs_trackball_r: now also U1.3 (PB14); no longer U1.10 (PA15)
- new net button_user_l: SW1.1, U2.26 (PA0)
- new net button_user_r: SW2.1, U1.26 (PA0)
- new net cs_user_l: J11.2 (Pin_2), U1.10 (PA15), U2.10 (PA15)
- new net cs_user_r: J12.2 (Pin_2)
- new net scl_l: U2.14 (PB6)
- no-connect marks 29 -> 34
Other:
- note added: "These buttons share the same pin as the on-board button. It is programmed in firmware to jump into STM32 dfu bootloader once pressed."
- moved on the sheet: J1, J10, J2, J3, J4, J5, J6, J7, J8, J9

Commit message: Release Candidate
Connections:
- net +3V3: now also U1.20 (3V3); no longer U1.38 (3V3)
- net cs_eeprom_l: now also U2.30 (PA4)
- net cs_eeprom_r: now also U1.30 (PA4)
- net cs_user_l: no longer U1.10 (PA15)
- net cs_user_r: now also U1.10 (PA15)
- net serial_r: now also U1.6 (PA9)
Changed lines of the file:
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@@
-(kicad_sch (version 20211123) (generator eeschema)
+(kicad_sch (version 20210621) (generator eeschema)
   (paper "A4")
   (title_block
@@
   (no_connect (at 142.875 168.275))
   (no_connect (at 163.195 160.655))
+  (no_connect (at 163.195 117.475))
   (no_connect (at 137.795 168.275))
   (no_connect (at 205.994 31.496))
-  (no_connect (at 163.83 35.052))
-  (no_connect (at 117.475 160.655))
+  (no_connect (at 163.83 34.925))
   (no_connect (at 118.11 37.465))
   (no_connect (at 163.83 42.545))
@@
     )
   )
-  (global_label "cs_eeprom_l" (shape input) (at 164.084 60.325 0)
-    (effects (font (size 1.27 1.27)) (justify left))
-    (property "Intersheet References" "${INTERSHEET_REFS}" (id 0) (at 168.5533 60.4044 0)
+  (global_label "cs_eeprom_l" (shape input) (at 163.83 60.325 0)
+    (effects (font (size 1.27 1.27)) (justify left))
+    (property "Intersheet References" "${INTERSHEET_REFS}" (id 0) (at 168.2993 60.4044 0)
       (effects (font (size 1.27 1.27)) (justify left) hide)
     )
@@
     )
   )
-  (global_label "cs_eeprom_r" (shape input) (at 163.449 137.795 0)
-    (effects (font (size 1.27 1.27)) (justify left))
-    (property "Intersheet References" "${INTERSHEET_REFS}" (id 0) (at 167.9183 137.8744 0)
+  (global_label "cs_eeprom_r" (shape input) (at 163.195 137.795 0)
+    (effects (font (size 1.27 1.27)) (justify left))
+    (property "Intersheet References" "${INTERSHEET_REFS}" (id 0) (at 167.6643 137.8744 0)
       (effects (font (size 1.27 1.27)) (justify left) hide)
     )
@@
     )
   )
-  (global_label "serial_r" (shape input) (at 117.094 125.095 180)
-    (effects (font (size 1.27 1.27)) (justify right))
-    (property "Intersheet References" "${INTERSHEET_REFS}" (id 0) (at 109.359 125.0156 0)
+  (global_label "serial_r" (shape input) (at 117.475 125.095 180)
+    (effects (font (size 1.27 1.27)) (justify right))
+    (property "Intersheet References" "${INTERSHEET_REFS}" (id 0) (at 109.74 125.0156 0)
       (effects (font (size 1.27 1.27)) (justify right) hide)
     )
@@
     )
   )
-  (global_label "cs_user_l" (shape input) (at 117.475 135.255 180)
+  (global_label "cs_user_r" (shape input) (at 117.475 135.255 180)
     (effects (font (size 1.27 1.27)) (justify right))
     (property "Intersheet References" "${INTERSHEET_REFS}" (id 0) (at 113.0057 135.1756 0)
@@
     (pin "1")
   )
-  (symbol (lib_id "power:+3.3V") (at 163.195 117.475 270) (unit 1)
-    (in_bom yes) (on_board yes)
-    (property "Reference" "#PWR0117" (id 0) (at 159.385 117.475 0)
-      (effects (font (size 1.27 1.27)) hide)
-    )
-    (property "Value" "+3.3V" (id 1) (at 165.735 117.475 90)
-      (effects (font (size 1.27 1.27)) (justify left))
-    )
-    (property "Footprint" "" (id 2) (at 163.195 117.475 0)
-      (effects (font (size 1.27 1.27)) hide)
-    )
-    (property "Datasheet" "" (id 3) (at 163.195 117.475 0)
-      (effects (font (size 1.27 1.27)) hide)
-    )
-    (pin "1")
-  )
   (symbol (lib_id "power:GND") (at 252.984 44.196 270) (unit 1)
     (in_bom yes) (on_board yes)
@@
     (pin "1")
     (pin "2")
+  )
+  (symbol (lib_id "power:+3.3V") (at 117.475 160.655 90) (unit 1)
+    (in_bom yes) (on_board yes)
+    (property "Reference" "#PWR0135" (id 0) (at 121.285 160.655 0)
+      (effects (font (size 1.27 1.27)) hide)
+    )
+    (property "Value" "+3.3V" (id 1) (at 114.935 160.655 90)
+      (effects (font (size 1.27 1.27)) (justify left))
+    )
+    (property "Footprint" "" (id 2) (at 117.475 160.655 0)
+      (effects (font (size 1.27 1.27)) hide)
+    )
+    (property "Datasheet" "" (id 3) (at 117.475 160.655 0)
+      (effects (font (size 1.27 1.27)) hide)
+    )
+    (pin "1")
   )
   (symbol (lib_id "Connector:Conn_01x06_Female") (at 278.13 123.825 0) (unit 1)
@@
       (reference "#PWR0116") (unit 1) (value "+5V") (footprint "")
     )
-    (path "/39a6cc12-820c-4bba-9063-3898a59c9c1e"
-      (reference "#PWR0117") (unit 1) (value "+3.3V") (footprint "")
-    )
     (path "/82adad32-0eb2-4a31-9983-6f031771039e"
       (reference "#PWR0118") (unit 1) (value "GND") (footprint "")
@@
       (reference "#PWR0134") (unit 1) (value "+5V") (footprint "")
     )
+    (path "/b9f037c6-265c-43b9-9fc1-ba6baf0e5ea3"
+      (reference "#PWR0135") (unit 1) (value "+3.3V") (footprint "")
+    )
     (path "/c86294cf-08bd-4fd0-9843-a692fca1caaf"

Commit message: Bugfix release 1.1
PB2 has a pulldown on the WeACT board to ensure BOOT1
is low during boot up. Otherwise jumping into the bootloader
is not ensured. So COL3 is moved from PB2 to PB10 as the pull
down prevents this pin from beeing used for matrix scanning.
Connections:
- net col3_l: now also U2.37 (PB10); no longer U2.36 (PB2)
- net col3_r: now also U1.37 (PB10); no longer U1.36 (PB2)
Changed lines of the file:
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@@
   (no_connect (at 135.255 168.275))
   (no_connect (at 117.475 112.395))
-  (no_connect (at 163.195 120.015))
   (no_connect (at 118.11 34.925))
+  (no_connect (at 163.195 122.555))
   (no_connect (at 117.475 114.935))
   (no_connect (at 163.195 158.115))
@@
   (no_connect (at 205.994 31.496))
   (no_connect (at 163.83 34.925))
+  (no_connect (at 163.83 45.085))
   (no_connect (at 118.11 37.465))
-  (no_connect (at 163.83 42.545))
   (no_connect (at 163.195 153.035))
   (no_connect (at 118.11 52.705))
@@
     )
   )
-  (global_label "col3_r" (shape input) (at 163.195 122.555 0)
-    (effects (font (size 1.27 1.27)) (justify left))
-    (property "Intersheet References" "${INTERSHEET_REFS}" (id 0) (at 192.405 161.925 0)
+  (global_label "col3_r" (shape input) (at 163.195 120.015 0)
+    (effects (font (size 1.27 1.27)) (justify left))
+    (property "Intersheet References" "${INTERSHEET_REFS}" (id 0) (at 192.405 159.385 0)
       (effects (font (size 1.27 1.27)) hide)
     )
@@
     )
   )
-  (global_label "col3_l" (shape input) (at 163.83 45.085 0)
-    (effects (font (size 1.27 1.27)) (justify left))
-    (property "Intersheet References" "${INTERSHEET_REFS}" (id 0) (at 193.04 84.455 0)
-      (effects (font (size 1.27 1.27)) hide)
-    )
+  (global_label "col3_l" (shape input) (at 163.83 42.545 0)
+    (effects (font (size 1.27 1.27)) (justify left))
+    (property "Intersheet References" "${INTERSHEET_REFS}" (id 0) (at 193.04 81.915 0)
+      (effects (font (size 1.27 1.27)) hide)
+    )

Commit message: Remove SPI user, add breakouts for audio and row 6
Parts:
- removed R3, R6: 5.1k, Resistor_SMD:R_1206_3216Metric_Pad1.30x1.75mm_HandSolder, symbol Device:R
- J11: value SPI user -> I2nc and audio
- J12: value SPI user -> I2C and audio
- J6, J9: footprint Library:5_PinHeader -> Library:6_PinHeader; symbol Connector:Conn_01x05_Female -> Connector:Conn_01x06_Female
- R1, R4, R5, R7: footprint Resistor_SMD:R_1206_3216Metric_Pad1.30x1.75mm_HandSolder -> Resistor_SMD:R_0805_2012Metric_Pad1.20x1.40mm_HandSolder
- R2, R8: value 5.1k -> 10k; footprint Resistor_SMD:R_1206_3216Metric_Pad1.30x1.75mm_HandSolder -> Resistor_SMD:R_0805_2012Metric_Pad1.20x1.40mm_HandSolder
Connections:
- net +5V: now also J11.4 (Pin_4), J12.4 (Pin_4); no longer J11.1 (Pin_1), J12.1 (Pin_1)
- net GND: now also J11.2 (Pin_2), J11.3 (Pin_3), J12.2 (Pin_2), J12.3 (Pin_3); no longer J11.6 (Pin_6), J12.6 (Pin_6)
- net col1_l: now also U2.13 (PB5); no longer U2.34 (PB0)
- net col1_r: now also U1.13 (PB5); no longer U1.34 (PB0)
- net col2_l: now also U2.12 (PB4); no longer U2.35 (PB1)
- net col2_r: now also U1.12 (PB4); no longer U1.35 (PB1)
- net col3_l: now also U2.4 (PB15); no longer U2.37 (PB10)
- net col3_r: now also U1.4 (PB15); no longer U1.37 (PB10)
- net col4_l: now also U2.3 (PB14); no longer U2.11 (PB3)
- net col4_r: now also U1.3 (PB14); no longer U1.11 (PB3)
- net col5_l: now also U2.10 (PA15); no longer U2.12 (PB4)
- net col5_r: now also U1.10 (PA15); no longer U1.12 (PB4)
- net col6_l: now also U2.5 (PA8); no longer U2.13 (PB5)
- net col6_r: now also U1.5 (PA8); no longer U1.13 (PB5)
- net cs_trackball_l: now also U2.34 (PB0); no longer U2.3 (PB14)
- net cs_trackball_r: now also U1.34 (PB0); no longer U1.3 (PB14)
- net dfu_bootloader_bodge_l: now also J10.6 (Pin_6)
- net dfu_bootloader_bodge_r: now also J8.6 (Pin_6); no longer U1.7 (PA10)
- net miso_l: no longer J11.5 (Pin_5)
- net miso_r: no longer J12.5 (Pin_5)
- net mosi_l: no longer J11.3 (Pin_3)
- net mosi_r: no longer J12.3 (Pin_3)
- net row1_l: now also U2.11 (PB3); no longer U2.4 (PB15)
- net row1_r: now also U1.11 (PB3); no longer U1.4 (PB15)
- net row2_l: now also U2.14 (PB6); no longer U2.28 (PA2)
- net row2_r: now also U1.14 (PB6); no longer U1.28 (PA2)
- net row3_l: now also U2.1 (PB12); no longer U2.16 (PB8)
- net row3_r: now also U1.1 (PB12); no longer U1.16 (PB8)
- net row4_l: now also U2.2 (PB13); no longer U2.5 (PA8)
- net row4_r: now also U1.2 (PB13); no longer U1.5 (PA8)
- net sck_l: no longer J11.4 (Pin_4)
- net sck_r: no longer J12.4 (Pin_4)
- net scl_l: now also J11.5 (Pin_5), U2.16 (PB8); no longer U2.14 (PB6)
- net scl_r: now also J12.5 (Pin_5), U1.16 (PB8); no longer U1.14 (PB6)
- net sda_l: now also J11.6 (Pin_6), U2.17 (PB9); no longer U2.15 (PB7)
- net sda_r: now also J12.6 (Pin_6), U1.17 (PB9); no longer U1.15 (PB7)
- net serial_l: now also U2.28 (PA2); no longer U2.6 (PA9)
- net serial_r: now also U1.29 (PA3); no longer U1.6 (PA9)
- net split_hand_l: now also U2.23 (PC14); no longer U2.29 (PA3)
- net split_hand_r: now also U1.23 (PC14); no longer U1.29 (PA3)
- net serial_rx_r: now reaches J1.S
- net serial_rx_r: now also U1.28 (PA2)
- net serial_rx_l: now reaches J2.S
- net serial_rx_l: now also U2.29 (PA3)
- net cs_eeprom_l: no longer names the net of U2.30 (PA4)
- net cs_eeprom_r: no longer names the net of U1.30 (PA4)
- removed net cs_user_l: J11.2 (Pin_2), U2.10 (PA15)
- removed net cs_user_r: J12.2 (Pin_2), U1.10 (PA15)
- removed net row5_l: J10.6 (Pin_6), U2.17 (PB9)
- removed net row5_r: J8.6 (Pin_6), U1.17 (PB9)
- new net audio_l: J11.1 (Pin_1), U2.35 (PB1)
- new net audio_r: J12.1 (Pin_1), U1.35 (PB1)
- new net row6_l: J9.6 (Pin_6), U2.15 (PB7)
- new net row6_r: J6.6 (Pin_6), U1.15 (PB7)
- no-connect marks 34 -> 30
Other:
- note removed: "Serial split comms in Half-duplex mode operate the TX pin in open drain configuration. Therefore a pull-up resistor is needed."
- moved on the sheet: J12, U1, U2
