File: adapter/adapter.kicad_sch (KiCad schematic)
At the start: 28 parts, among them J1 Serial, J10 Ribbon, J11 SPI user, J12 SPI user, J2 Serial, J3 RGB, J4 RGB, J5 Trackball, J6 Ribbon, J7 Trackball, J8 Ribbon, J9 Ribbon, SW1 USER, SW2 USER, U1 STM32F401 / STM32F411 Blackpi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, U2 STM32F401 / STM32F411 Blackpi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

Commit message: Start rev1.2 and move update button 3.75mm up
Other:
- company: Bastardkb x KarlK90 -> BastardKB x KarlK90
Changed lines of the file:
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@@
-(kicad_sch (version 20210621) (generator eeschema)
+(kicad_sch (version 20211123) (generator eeschema)
   (paper "A4")
   (title_block
     (title "Charybdis Blackpill Holder")
-    (date "2021-12-02")
-    (rev "0.1")
-    (company "Bastardkb x KarlK90")
+    (date "2022-01-20")
+    (rev "1.2")
+    (company "BastardKB x KarlK90")
     (comment 1 "Licensed under CERN-OHL-W v2")
   )

Commit message: Add I2C header to schematic, start placement
Parts:
- added J13, J14: I2C, Library:4_PinHeader, symbol Connector:Conn_01x04_Female
- added R10, R11, R12, R9: 5.1k, Resistor_SMD:R_1206_3216Metric_Pad1.30x1.75mm_HandSolder, symbol Device:R
Connections:
- net +5V: now also J13.1 (Pin_1), J14.1 (Pin_1), R10.1, R11.1, R12.1, R9.1
- net GND: now also J13.4 (Pin_4), J14.4 (Pin_4)
- net scl_l: now also R11.2
- net scl_r: now also J13.2 (Pin_2), J14.2 (Pin_2), R9.2
- net sda_l: now also R12.2
- net sda_r: now also J13.3 (Pin_3), J14.3 (Pin_3), R10.2
Other:
- note added: "I2C bus operates in open drain configuration. Therefore pull-up resistors on clock (SCL) and data (SDA) is needed."
