File: adapter/adapter.kicad_pcb (KiCad board)
At the start: 2 copper layers, 93.8 x 42.3 mm, 16 parts, among them J1 AudioJack4, J2 AudioJack4, J3 Conn_01x02_Female, J4 Conn_01x03_Female, J5 Conn_01x03_Female, J6 Conn_01x02_Female, J7 Conn_01x06_Female, J9 Conn_01x06_Female, SW1 SW_SPST, SW2 SW_SPST, U2 eliteC, U3 YAAJ_WeAct_BlackPill_Part_Lik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

Commit message: Update schematic for left and right hand
Parts:
- removed SW1, SW2: SW_SPST, customs:switch_rst
- removed U3: YAAJ_WeAct_BlackPill_Part_Like_SWD_Breakout, Library:YAAJ_WeAct_BlackPill_SWD_2
- added J10: Ribbon, Connector_PinHeader_2.54mm:PinHeader_1x06_P2.54mm_Vertical, F.Cu at (65.2, 35.7)
- added J8: Ribbon, Connector_PinHeader_2.54mm:PinHeader_1x06_P2.54mm_Vertical, F.Cu at (102.6, 56.0)
- added R1: 5.1k, Resistor_SMD:R_0805_2012Metric_Pad1.20x1.40mm_HandSolder, F.Cu at (107.6, 42.9)
- added R2: 5.1k, Resistor_SMD:R_0805_2012Metric_Pad1.20x1.40mm_HandSolder, F.Cu at (83.4, 62.6)
- added R3: 5.1k, Resistor_SMD:R_0805_2012Metric_Pad1.20x1.40mm_HandSolder, F.Cu at (83.3, 57.7)
- added R4: 5.1k, Resistor_SMD:R_0805_2012Metric_Pad1.20x1.40mm_HandSolder, F.Cu at (83.4, 59.8)
- added R5: 5.1k, Resistor_SMD:R_0805_2012Metric_Pad1.20x1.40mm_HandSolder, F.Cu at (35.4, 60.2)
- added R6: 5.1k, Resistor_SMD:R_0805_2012Metric_Pad1.20x1.40mm_HandSolder, F.Cu at (35.1, 63.1)
- added R7: 5.1k, Resistor_SMD:R_0805_2012Metric_Pad1.20x1.40mm_HandSolder, F.Cu at (39.4, 42.5)
- added R8: 5.1k, Resistor_SMD:R_0805_2012Metric_Pad1.20x1.40mm_HandSolder, F.Cu at (38.7, 64.8)
- added U1: STM32F401 / STM32F411 Blackpill Breakout, Library:YAAJ_WeAct_BlackPill_SWD_2, B.Cu at (60.8, 32.9)
- J1, J2: value AudioJack4 -> Serial
- J3: value Conn_01x02_Female -> RGB; footprint Connector_PinSocket_2.54mm:PinSocket_2x01_P2.54mm_Vertical -> Connector_PinSocket_2.54mm:PinSocket_1x03_P2.54mm_Vertical
- J4: value Conn_01x03_Female -> RGB
- J5: value Conn_01x03_Female -> Trackball; footprint Connector_PinSocket_2.54mm:PinSocket_1x03_P2.54mm_Vertical -> Connector_PinHeader_2.54mm:PinHeader_1x06_P2.54mm_Vertical
- J6: value Conn_01x02_Female -> Ribbon; footprint Connector_PinSocket_2.54mm:PinSocket_2x01_P2.54mm_Vertical -> Connector_PinHeader_2.54mm:PinHeader_1x06_P2.54mm_Vertical
- J7: value Conn_01x06_Female -> Trackball
- J9: value Conn_01x06_Female -> Ribbon
- U2: value eliteC -> STM32F401 / STM32F411 Blackpill Breakout; footprint Library:Elite-C-castellated-29pin-holes -> Library:YAAJ_WeAct_BlackPill_SWD_2; moved to F.Cu
- moved U2 62.7 mm to (83.7, 32.8), turned to 0 degrees
- moved G*** 51.1 mm to (73.6, 67.2)
- moved G*** 51.1 mm to (73.7, 67.2)
- moved G*** 51.1 mm to (95.8, 38.1)
- moved J1 51.1 mm to (38.8, 38.2)
- moved J2 51.1 mm to (114.2, 38.3)
- moved J3 51.1 mm to (35.3, 46.9)
- moved J4 51.1 mm to (35.3, 49.7)
- moved J6 51.1 mm to (112.2, 47.0)
- moved J9 51.1 mm to (106.8, 47.2)
- moved G*** 51.1 mm to (51.7, 38.1)
- moved J7 51.1 mm to (40.9, 47.3)
- moved J5 51.1 mm to (112.2, 49.7)
Connections:
- J1 pad R1: Gnd -> GND
- J1 pad R2: Net-(J1-PadR2) -> serial_r
- J1 pad T: Vcc -> +5V
- J2 pad R1: Gnd2 -> GND
- J2 pad R2: Net-(J2-PadR2) -> serial_l
- J2 pad T: Vcc2 -> +5V
- J3 pad 1: Net-(J3-Pad1) -> +5V
- J3 pad 2: Net-(J3-Pad2) -> GND
- J4 pad 1: Vcc -> +5V
- J4 pad 2: Gnd -> GND
- J4 pad 3: Din -> rgb_r
- J5 pad 1: Vcc2 -> +5V
- J5 pad 2: Gnd2 -> ss_trackball_l
- J5 pad 3: Din2 -> mosi_l
- J6 pad 1: Net-(J6-Pad1) -> unconnected-(J6-Pad1)
- J6 pad 2: Net-(J6-Pad2) -> unconnected-(J6-Pad2)
- J7 pad 1: Vcc -> +5V
- J7 pad 2: ss -> ss_trackball_r
- J7 pad 3: mosi -> mosi_r
- J7 pad 4: sc -> sck_r
- J7 pad 5: miso -> miso_r
- J7 pad 6: Gnd -> GND
- J9 pad 1: Vcc2 -> row4_l
- J9 pad 2: ss2 -> row3_l
- J9 pad 3: mosi2 -> col4_l
- J9 pad 4: sc2 -> col5_l
- J9 pad 5: miso2 -> col6_l
- J9 pad 6: Gnd2 -> row5_l
- U2 pad 1: Din2 -> row1_l
- U2 pad 10: unconnected-(U2-Pad10) -> ss_trackball_l
- U2 pad 11: unconnected-(U2-Pad11) -> col4_l
- U2 pad 12: unconnected-(U2-Pad12) -> col5_l
- U2 pad 13: unconnected-(U2-Pad13) -> col6_l
- U2 pad 14: mosi2 -> row5_l
- U2 pad 15: miso2 -> unconnected-(U2-Pad15)
- U2 pad 16: sc2 -> unconnected-(U2-Pad16)
- U2 pad 18: unconnected-(U2-Pad18) -> +5V
- U2 pad 19: unconnected-(U2-Pad19) -> GND
- U2 pad 2: Net-(J2-PadR2) -> row2_l
- U2 pad 20: unconnected-(U2-Pad20) -> +3V3
- U2 pad 21: Vcc2 -> unconnected-(U2-Pad21)
- U2 pad 22: Rst2 -> unconnected-(U2-Pad22)
- U2 pad 23: Gnd2 -> unconnected-(U2-Pad23)
- U2 pad 24: ss2 -> unconnected-(U2-Pad24)
- U2 pad 26: unconnected-(U2-Pad26) -> split_hand_l
- U2 pad 27: unconnected-(U2-Pad27) -> rgb_l
- U2 pad 3: Gnd2 -> row3_l
- U2 pad 4: Gnd2 -> row4_l
- U2 pad 5: Net-(J6-Pad2) -> unconnected-(U2-Pad5)
- U2 pad 6: Net-(J6-Pad1) -> unconnected-(U2-Pad6)
- U2 pad 7: unconnected-(U2-Pad7) -> dfu_bootloader_bodge_l
Routing:
- net Vcc2: track 98.1 -> 0.00 mm
- net Gnd2: track 80.1 -> 0.00 mm, vias 2 -> 0
- net Gnd: track 64.2 -> 0.00 mm, vias 1 -> 0
- net miso2: track 52.4 -> 0.00 mm
- net sc2: track 41.4 -> 0.00 mm
- net Net-(J1-PadR2): track 36.6 -> 0.00 mm, vias 1 -> 0
- net mosi2: track 36.0 -> 0.00 mm
- net Din: track 35.2 -> 0.00 mm
- net Din2: track 32.9 -> 0.00 mm
- net ss: track 29.8 -> 0.00 mm
- net ss2: track 29.5 -> 0.00 mm
- net Net-(J3-Pad1): track 25.8 -> 0.00 mm, vias 1 -> 0
- net Net-(J3-Pad2): track 25.1 -> 0.00 mm, vias 1 -> 0
- net Rst: track 23.9 -> 0.00 mm, vias 2 -> 0
- net Vcc: track 21.7 -> 0.00 mm
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- added copper zone on B.Cu, net GND
- added copper zone on F.Cu, net GND
- removed copper zone on B.Cu, net Gnd
- removed copper zone on F.Cu, net Gnd
- removed copper zone on B.Cu, net Gnd2
- removed copper zone on F.Cu, net Gnd2
Other:
- outline, holes or cut-outs redrawn
- board text removed: "RST"

Commit message: component placement
Parts:
- removed J10, J6, J8: Ribbon, Connector_PinHeader_2.54mm:PinHeader_1x06_P2.54mm_Vertical
- removed J3, J4: RGB, Connector_PinSocket_2.54mm:PinSocket_1x03_P2.54mm_Vertical
- removed J5: Trackball, Connector_PinHeader_2.54mm:PinHeader_1x06_P2.54mm_Vertical
- removed R1, R2, R3, R4, R5, R6, R7, R8: 5.1k, Resistor_SMD:R_0805_2012Metric_Pad1.20x1.40mm_HandSolder
- added J2: Serial, Library:Jack_3.5mm_PJ320E_Horizontal, F.Cu at (171.2, 24.6)
- added REF**: MountingHole_4mm_Pad, MountingHole:MountingHole_4mm_Pad, F.Cu at (116.0, 25.2)
- added REF**: MountingHole_4mm_Pad, MountingHole:MountingHole_4mm_Pad, F.Cu at (132.2, 25.2)
- added REF**: MountingHole_4mm_Pad, MountingHole:MountingHole_4mm_Pad, F.Cu at (81.4, 53.1)
- added REF**: MountingHole_4mm_Pad, MountingHole:MountingHole_4mm_Pad, F.Cu at (166.7, 53.0)
- J2: value Serial -> AudioJack4
- J9: value Ribbon -> Conn_01x06_Female
- U1: moved to F.Cu
- moved U2 55.8 mm to (138.6, 23.1)
- moved G*** 51.1 mm to (123.9, 58.3)
- moved G*** 51.1 mm to (124.0, 58.3)
- moved G*** 51.1 mm to (146.1, 29.2)
- moved J1 51.1 mm to (89.1, 29.3)
- moved J2 51.1 mm to (164.5, 29.4)
- moved J9 51.1 mm to (157.1, 38.4)
- moved G*** 51.1 mm to (102.0, 29.2)
- moved J7 51.1 mm to (91.2, 38.4)
- moved U1 35.1 mm to (94.5, 23.1), turned to 0 degrees
Connections:
- J2 pad R1: GND -> Gnd2
- J2 pad R2: serial_l -> Net-(J2-PadR2)
- J2 pad T: +5V -> Vcc2
- J9 pad 1: row4_l -> Vcc2
- J9 pad 2: row3_l -> ss2
- J9 pad 3: col4_l -> mosi2
- J9 pad 4: col5_l -> sc2
- J9 pad 5: col6_l -> miso2
- J9 pad 6: row5_l -> Gnd2
Routing:
- added copper zone on B.Cu, net Gnd2
- added copper zone on F.Cu, net Gnd2
Other:
- outline, holes or cut-outs redrawn
- board text added: "todo - version number - check onboard buttons are accessible - check edge cuts - change board name"

Commit message: edge cuts
Parts:
- moved J7 101.8 mm to (192.4, 49.3)
- moved J9 19.8 mm to (176.5, 42.5)
- moved U1 1.00 mm to (93.5, 23.1)
- moved U2 1.00 mm to (139.6, 23.1)
Other:
- board size 93.8 x 42.3 mm -> 42.2 x 67.2 mm

Commit message: move blackpill, better edge cuts
Parts:
- moved U1 2.54 mm to (93.5, 20.6)
- moved U2 2.54 mm to (139.6, 20.5)
Other:
- board size 42.2 x 67.2 mm -> 42.3 x 67.2 mm

Commit message: flip blackpill
Parts:
- U1, U2: moved to B.Cu
- moved U2 15.2 mm to (154.9, 20.5), turned to 180 degrees
- moved U1 15.2 mm to (108.8, 20.6), turned to 180 degrees

Commit message: place headers
Parts:
- added J10: Ribbon, Connector_PinHeader_2.54mm:PinHeader_1x06_P2.54mm_Vertical, F.Cu at (135.4, 55.0)
- added J3: RGB, Connector_PinSocket_2.54mm:PinSocket_1x03_P2.54mm_Vertical, F.Cu at (218.1, 55.2)
- added J4: RGB, Connector_PinSocket_2.54mm:PinSocket_1x03_P2.54mm_Vertical, F.Cu at (222.7, 55.2)
- added J5: Trackball, Connector_PinHeader_2.54mm:PinHeader_1x06_P2.54mm_Vertical, F.Cu at (140.8, 73.8)
- added J8: Ribbon, Connector_PinHeader_2.54mm:PinHeader_1x06_P2.54mm_Vertical, F.Cu at (213.5, 55.2)
- added R1: 5.1k, Resistor_SMD:R_0805_2012Metric_Pad1.20x1.40mm_HandSolder, F.Cu at (227.4, 54.3)
- added R2: 5.1k, Resistor_SMD:R_0805_2012Metric_Pad1.20x1.40mm_HandSolder, F.Cu at (227.4, 60.2)
- added R3: 5.1k, Resistor_SMD:R_0805_2012Metric_Pad1.20x1.40mm_HandSolder, F.Cu at (218.2, 64.0)
- added R4: 5.1k, Resistor_SMD:R_0805_2012Metric_Pad1.20x1.40mm_HandSolder, F.Cu at (222.9, 64.0)
- added R5: 5.1k, Resistor_SMD:R_0805_2012Metric_Pad1.20x1.40mm_HandSolder, F.Cu at (227.4, 57.3)
- added R6: 5.1k, Resistor_SMD:R_0805_2012Metric_Pad1.20x1.40mm_HandSolder, F.Cu at (232.1, 54.3)
- added R7: 5.1k, Resistor_SMD:R_0805_2012Metric_Pad1.20x1.40mm_HandSolder, F.Cu at (218.2, 67.0)
- added R8: 5.1k, Resistor_SMD:R_0805_2012Metric_Pad1.20x1.40mm_HandSolder, F.Cu at (232.1, 57.3)
- moved J7 101.0 mm to (94.3, 73.6), turned to 90 degrees
- moved J9 41.3 mm to (135.6, 37.0)

Commit message: component placement
Parts:
- removed J9: Conn_01x06_Female, Connector_PinHeader_2.54mm:PinHeader_1x06_P2.54mm_Vertical
- added J6: Ribbon, Connector_PinHeader_2.54mm:PinHeader_1x05_P2.54mm_Vertical, F.Cu at (149.3, 73.2)
- moved R2 84.1 mm to (144.3, 46.8)
- moved R1 82.5 mm to (146.0, 40.2)
- moved R4 75.0 mm to (150.9, 43.1)
- moved R3 71.8 mm to (147.9, 49.0)
- moved J4 63.2 mm to (161.6, 39.0)
- moved J10 20.0 mm to (143.7, 73.2)
- moved J5 18.8 mm to (155.4, 85.7), turned to 180 degrees
Other:
- outline, holes or cut-outs redrawn
- board text added: "BLACKPILL HOLDER 0.1"
- board text added: "C1"
- board text added: "C2"
- board text added: "C3"
- board text added: "C4"
- board text added: "C5"
- board text added: "C6"
- board text added: "R1"
- board text added: "R2"
- board text added: "R3"
- board text added: "R4"
- board text added: "R5"

Commit message: component placement
Parts:
- R1, R2, R3, R4: footprint Resistor_SMD:R_0805_2012Metric_Pad1.20x1.40mm_HandSolder -> Resistor_SMD:R_1206_3216Metric_Pad1.30x1.75mm_HandSolder; moved to B.Cu
- R5, R6, R7, R8: footprint Resistor_SMD:R_0805_2012Metric_Pad1.20x1.40mm_HandSolder -> Resistor_SMD:R_1206_3216Metric_Pad1.30x1.75mm_HandSolder
- moved R4 10.2 mm to (144.4, 50.9), turned to 180 degrees
- moved R1 8.53 mm to (150.3, 47.6), turned to 180 degrees
- moved R3 3.07 mm to (150.3, 50.9), turned to 180 degrees
- moved R2 0.79 mm to (144.4, 47.6), turned to 180 degrees
