File: adapter/adapter.kicad_pcb (KiCad board)
At the start: 2 copper layers, 42.3 x 67.2 mm, 28 parts, among them J1 Serial, J10 Ribbon, J2 AudioJack4, J2 Serial, J3 RGB, J4 RGB, J5 Trackball, J6 Ribbon, J7 Trackball, J8 Ribbon, U1 STM32F401 / STM32F411 Blackpi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, U2 STM32F401 / STM32F411 Blackpi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

Commit message: placement
Parts:
- removed the J2 at (171.2, 24.6)
- moved G*** 45.2 mm to (191.3, 27.8)
- moved J5 12.7 mm to (155.4, 73.0), turned to 0 degrees
Other:
- outline, holes or cut-outs redrawn
Changed lines of the file:
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@@
   )
   (footprint "Connector_PinHeader_2.54mm:PinHeader_1x06_P2.54mm_Vertical" (layer "F.Cu")
-    (at 155.41 85.65 180)
+    (at 155.45 72.99)
     (descr "Through hole straight pin header, 1x06, 2.54mm pitch, single row")
     (tags "Through hole pin header THT 1x06 2.54mm single row")
@@
     (fp_line (start -1.27 13.97) (end -1.27 -0.635) (layer "F.Fab") (width 0.1))
     (fp_line (start 1.27 -1.27) (end 1.27 13.97) (layer "F.Fab") (width 0.1))
-    (pad "1" thru_hole rect (at 0 0 180) (size 1.7 1.7) (drill 1) (layers *.Cu *.Mask)
+    (pad "1" thru_hole rect (at 0 0) (size 1.7 1.7) (drill 1) (layers *.Cu *.Mask)
       (net 20 "+5V") (pinfunction "Pin_1") (pintype "passive"))
-    (pad "2" thru_hole oval (at 0 2.54 180) (size 1.7 1.7) (drill 1) (layers *.Cu *.Mask)
+    (pad "2" thru_hole oval (at 0 2.54) (size 1.7 1.7) (drill 1) (layers *.Cu *.Mask)
       (net 71 "ss_trackball_l") (pinfunction "Pin_2") (pintype "passive"))
-    (pad "3" thru_hole oval (at 0 5.08 180) (size 1.7 1.7) (drill 1) (layers *.Cu *.Mask)
+    (pad "3" thru_hole oval (at 0 5.08) (size 1.7 1.7) (drill 1) (layers *.Cu *.Mask)
       (net 68 "mosi_l") (pinfunction "Pin_3") (pintype "passive"))
-    (pad "4" thru_hole oval (at 0 7.62 180) (size 1.7 1.7) (drill 1) (layers *.Cu *.Mask)
+    (pad "4" thru_hole oval (at 0 7.62) (size 1.7 1.7) (drill 1) (layers *.Cu *.Mask)
       (net 70 "sck_l") (pinfunction "Pin_4") (pintype "passive"))
-    (pad "5" thru_hole oval (at 0 10.16 180) (size 1.7 1.7) (drill 1) (layers *.Cu *.Mask)
+    (pad "5" thru_hole oval (at 0 10.16) (size 1.7 1.7) (drill 1) (layers *.Cu *.Mask)
       (net 69 "miso_l") (pinfunction "Pin_5") (pintype "passive"))
-    (pad "6" thru_hole oval (at 0 12.7 180) (size 1.7 1.7) (drill 1) (layers *.Cu *.Mask)
+    (pad "6" thru_hole oval (at 0 12.7) (size 1.7 1.7) (drill 1) (layers *.Cu *.Mask)
       (net 18 "GND") (pinfunction "Pin_6") (pintype "passive"))
     (model "${KICAD6_3DMODEL_DIR}/Connector_PinHeader_2.54mm.3dshapes/PinHeader_1x06_P2.54mm_Vertical.wrl" hide
@@
     )
   )
-  (footprint "Library:Jack_3.5mm_PJ320E_Horizontal" (layer "F.Cu")
-    (at 171.25 24.6)
-    (descr "Headphones with microphone connector, 3.5mm, 4 pins (http://www.qingpu-electronics.com/en/products/WQP-PJ320E-177.html)")
-    (tags "3.5mm jack mic microphone phones headphones 4pins audio plug")
-    (property "JLCPCB BOM" "0")
-    (property "JLCPCB Part" "")
-    (property "Sheetfile" "adapter.kicad_sch")
-    (property "Sheetname" "")
-    (attr through_hole)
-    (fp_text reference "J2" (at 2.54 -13.97) (layer "F.SilkS") hide
-      (effects (font (size 1 1) (thickness 0.15)))
-    )
-    (fp_text value "Serial" (at 2.54 5.08) (layer "F.Fab")
-      (effects (font (size 1 1) (thickness 0.15)))
-    )
-    (fp_text user "${REFERENCE}" (at 2.54 -13.97) (layer "F.Fab")
-      (effects (font (size 1 1) (thickness 0.15)))
-    )
-    (fp_line (start 5.2 -9.3) (end 5.2 -12.1) (layer "F.SilkS") (width 0.12))
-    (fp_line (start -0.9 2.8) (end 3.7 2.8) (layer "F.SilkS") (width 0.12))
-    (fp_line (start 6.4 -9.3) (end 6.4 2.8) (layer "F.SilkS") (width 0.12))
-    (fp_line (start 5.2 -9.3) (end 6.4 -9.3) (layer "F.SilkS") (width 0.12))
-    (fp_line (start 5.2 -12.1) (end -0.6 -12.1) (layer "F.SilkS") (width 0.12))
-    (fp_line (start 6.4 2.8) (end 3.7 2.8) (layer "F.SilkS") (width 0.12))
-    (fp_line (start -0.6 -9.3) (end -0.6 -12.1) (layer "F.SilkS") (width 0.12))
-    (fp_line (start -0.9 -9.3) (end -0.9 2.8) (layer "F.SilkS") (width 0.12))
-    (fp_line (start -0.9 -9.3) (end -0.6 -9.3) (layer "F.SilkS") (width 0.12))
-    (fp_line (start 6.8 -12.5) (end 6.8 3) (layer "F.CrtYd") (width 0.05))
-    (fp_line (start -1.3 -12.5) (end 6.8 -12.5) (layer "F.CrtYd") (width 0.05))
-    (fp_line (start -1.3 -12.5) (end -1.3 3) (layer "F.CrtYd") (width 0.05))
-    (fp_line (start -1.3 3) (end 6.8 3) (layer "F.CrtYd") (width 0.05))
-    (fp_line (start -0.8 -9.2) (end -0.5 -9.2) (layer "F.Fab") (width 0.1))
-    (fp_line (start -0.5 -12) (end 5.1 -12) (layer "F.Fab") (width 0.1))
-    (fp_line (start 6.3 2) (end 5.3 2) (layer "F.Fab") (width 0.1))
-    (fp_line (start 5.1 -9.2) (end 6.3 -9.2) (layer "F.Fab") (width 0.1))
-    (fp_line (start 6.3 -9.2) (end 6.3 2) (layer "F.Fab") (width 0.1))
-    (fp_line (start -0.5 -9.2) (end -0.5 -12) (layer "F.Fab") (width 0.1))
-    (fp_line (start 3.7 2) (end -0.8 2) (layer "F.Fab") (width 0.1))
-    (fp_line (start 5.1 -12) (end 5.1 -9.2) (layer "F.Fab") (width 0.1))
-    (fp_line (start -0.8 2) (end -0.8 -9.2) (layer "F.Fab") (width 0.1))
-    (fp_circle (center 0.9 0) (end 1.2 0.15) (layer "F.Fab") (width 0.12) (fill none))
-    (pad "" thru_hole oval locked (at 5.5 -7 270) (size 2 1.4) (drill oval 1.2 0.6) (layers *.Cu *.Mask))
-    (pad "" np_thru_hole oval locked (at 2.3 -1.6 270) (size 1.5 1.5) (drill oval 1.5) (layers *.Cu *.Mask))
-    (pad "" np_thru_hole oval locked (at 2.3 -8.6 270) (size 1.5 1.5) (drill oval 1.5) (layers *.Cu *.Mask))
-    (pad "R1" thru_hole oval locked (at 0 -4 270) (size 2 1.4) (drill oval 1.2 0.6) (layers *.Cu *.Mask)
-      (net 18 "GND") (pintype "passive"))
-    (pad "R2" thru_hole oval locked (at 0 -7 270) (size 2 1.4) (drill oval 1.2 0.6) (layers *.Cu *.Mask)
-      (net 21 "serial_l") (pintype "passive"))
-    (pad "S" thru_hole oval locked (at 4.5 0.75 270) (size 3.5 1.4) (drill oval 2.7 0.6) (layers *.Cu *.Mask)
-      (net 5 "unconnected-(J2-PadS)") (pintype "passive+no_connect"))
-    (pad "T" thru_hole rect locked (at 0 0 270) (size 2 1.4) (drill oval 1.2 0.6) (layers *.Cu *.Mask)
-      (net 20 "+5V") (pintype "passive"))
-    (model "${KISYS3DMOD}/Connector_Audio.3dshapes/Jack_3.5mm_PJ320E_Horizontal.wrl"
-      (offset (xyz 0 0 0))
-      (scale (xyz 1 1 1))
-      (rotate (xyz 0 0 0))
-    )
-  )
   (footprint "MountingHole:MountingHole_4mm_Pad" (layer "F.Cu")
     (at 166.716 52.98)
@@
   )
   (footprint "LOGO" (layer "B.Cu")
-    (at 146.131301 29.22 180)
+    (at 191.32 27.83 180)
     (attr board_only exclude_from_pos_files exclude_from_bom)
     (fp_text reference "G***" (at 0 0) (layer "B.SilkS") hide
@@
   (gr_line (start 158.688078 59.871325) (end 158.688078 84.155026) (layer "Edge.Cuts") (width 0.2))
   (gr_line (start 139.207721 21.766283) (end 132.2 21.766283) (layer "Edge.Cuts") (width 0.2))
-  (gr_line (start 142.276572 54.46369) (end 142.276572 63.615026) (layer "Edge.Cuts") (width 0.2))
   (gr_line (start 161.228078 57.331325) (end 166.718015 57.331325) (layer "Edge.Cuts") (width 0.2))
   (gr_line (start 160.668073 20.920396) (end 157.451505 20.926952) (layer "Edge.Cuts") (width 0.2))
@@
   (gr_circle (center 166.774935 53.14027) (end 168.924935 53.14027) (layer "Edge.Cuts") (width 0.2) (fill none))
   (gr_arc (start 153.207721 23.766283) (mid 153.793507 22.352069) (end 155.207721 21.766283) (layer "Edge.Cuts") (width 0.2))
-  (gr_line (start 151.671087 63.615026) (end 151.671087 54.46369) (layer "Edge.Cuts") (width 0.2))
-  (gr_line (start 142.276572 63.615026) (end 151.671087 63.615026) (layer "Edge.Cuts") (width 0.2))
-  (gr_line (start 151.671087 54.46369) (end 142.276572 54.46369) (layer "Edge.Cuts") (width 0.2))
   (gr_line (start 164.892713 20.911785) (end 162.146796 20.917382) (layer "Edge.Cuts") (width 0.2))
   (gr_arc (start 139.207721 21.766283) (mid 140.621935 22.352069) (end 141.207721 23.766283) (layer "Edge.Cuts") (width 0.2))
@@
     (polygon
       (pts
-        (xy 176.385 68.295)
-        (xy 138.34 68.71)
-        (xy 129.89 39.54)
+        (xy 177.44 95.4)
+        (xy 128.78 93.16)
+        (xy 127.32 39.73)
         (xy 126.865 20.735)
         (xy 174.605 18.865)
@@
       36ae8b5e-208f-4981-b689-8bbeeb1e7a61
       3ce69f83-56f2-4a87-9f13-f82b2b8f1ebc
-      3d340bf4-bf18-451d-9794-48b05be14313
       5766e482-e474-44dd-b64d-a92c974904b7
       5a9d60f1-8eb2-49ef-9487-c1b847be82be
@@
       b7410a7b-73cc-4b71-887e-fe2fb58e7292
       b9c3a055-054e-4743-9e95-28a593ef6d9f
-      c7592407-d0a2-49b9-bcfe-711558139c4a
-      db7de36d-6618-4fca-9cd7-aea7b66156f9
-      e101acdb-3367-4990-96d3-0d88fede9b34
       e6fd80b0-5efd-4549-ab5d-27e87441e2cb
       eb6fd09a-901c-443e-9c1e-f568c4ca200b

Commit message: right edge cuts
Parts:
- added J9: Ribbon, Connector_PinHeader_2.54mm:PinHeader_1x05_P2.54mm_Vertical, F.Cu at (149.2, 73.2)
- moved J8 110.6 mm to (104.4, 73.2)
- moved J6 50.6 mm to (98.7, 73.2)
- moved J7 1.39 mm to (93.0, 73.2), turned to 0 degrees
Connections:
- U2 pad 40: +5V -> unconnected-(U2-Pad40)
Other:
- board size 42.3 x 67.2 mm -> 93.9 x 67.3 mm

Commit message: Traces for left side
Parts:
- removed REF** (x4): MountingHole_4mm_Pad, MountingHole:MountingHole_4mm_Pad
- added H1: M4, Library:MountingHole_4mm_Pad_Thin, F.Cu at (116.0, 25.2)
- added H2: M4, Library:MountingHole_4mm_Pad_Thin, F.Cu at (81.4, 53.1)
- added H3: M4, Library:MountingHole_4mm_Pad_Thin, F.Cu at (132.2, 25.2)
- added H4: M4, Library:MountingHole_4mm_Pad_Thin, F.Cu at (166.8, 53.1)
- added J11: SPI user, Library:6_PinHeader, F.Cu at (149.9, 73.5)
- added J12: SPI user, Library:6_PinHeader, F.Cu at (104.8, 73.8)
- added SW1: USER, Library:PushSwitch, B.Cu at (147.2, 64.9)
- added SW2: USER, Library:PushSwitch, B.Cu at (101.2, 64.9)
- J10, J5, J7, J8: footprint Connector_PinHeader_2.54mm:PinHeader_1x06_P2.54mm_Vertical -> Library:6_PinHeader
- J2: value AudioJack4 -> Serial
- J3: renamed from J4; footprint Connector_PinSocket_2.54mm:PinSocket_1x03_P2.54mm_Vertical -> Library:3_PinSocket
- J4: renamed from J3; footprint Connector_PinSocket_2.54mm:PinSocket_1x03_P2.54mm_Vertical -> Library:3_PinSocket
- J6, J9: footprint Connector_PinHeader_2.54mm:PinHeader_1x05_P2.54mm_Vertical -> Library:5_PinHeader
- R5, R6, R7, R8: moved to B.Cu
- U1, U2: footprint Library:YAAJ_WeAct_BlackPill_SWD_2 -> Library:WeAct_BlackPill_without_SWD_First_Row
- moved R5 141.3 mm to (86.4, 48.5), turned to 90 degrees
- moved R6 134.7 mm to (97.9, 42.3), turned to 180 degrees
- moved R8 134.7 mm to (97.9, 45.3), turned to 180 degrees
- moved J4 132.8 mm to (86.3, 39.0)
- moved R7 118.8 mm to (100.5, 50.4), turned to 180 degrees
- moved G*** 50.3 mm to (147.2, 52.0)
- moved G*** 22.8 mm to (101.2, 52.0)
- moved R4 17.5 mm to (161.8, 48.8), turned to 90 degrees
- moved R3 8.67 mm to (151.3, 42.3), turned to 90 degrees
- moved R1 6.15 mm to (147.3, 42.3), turned to 90 degrees
- moved R2 5.44 mm to (143.3, 42.3), turned to 90 degrees
- moved J10 5.07 mm to (138.7, 73.5)
- moved J9 4.95 mm to (144.3, 73.5)
- moved J8 4.42 mm to (108.8, 73.5)
- moved J6 2.49 mm to (101.2, 73.5)
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Connections:
- J2 pad R1: Gnd2 -> GND
- J2 pad R2: Net-(J2-PadR2) -> serial_l
- J2 pad T: Vcc2 -> +5V
- J3 pad 3: rgb_r -> rgb_l
- J4 pad 3: rgb_l -> rgb_r
- J5 pad 2: ss_trackball_l -> cs_trackball_l
- J7 pad 2: ss_trackball_r -> cs_trackball_r
- U1 pad 10: ss_trackball_r -> cs_user_l
- U1 pad 14: unconnected-(U1-Pad14) -> scl_r
- U1 pad 15: unconnected-(U1-Pad15) -> sda_r
- U1 pad 16: unconnected-(U1-Pad16) -> row3_r
- U1 pad 17: unconnected-(U1-Pad17) -> row5_r
- U1 pad 2: row2_r -> unconnected-(U1-Pad2)
- U1 pad 20: +3V3 -> unconnected-(U1-Pad20)
- U1 pad 26: split_hand_r -> button_user_r
- U1 pad 28: unconnected-(U1-Pad28) -> row2_r
- U1 pad 29: unconnected-(U1-Pad29) -> split_hand_r
- U1 pad 3: row3_r -> cs_trackball_r
- U1 pad 38: unconnected-(U1-Pad38) -> +3V3
- U1 pad 4: row4_r -> row1_r
- U1 pad 5: row5_r -> row4_r
- U2 pad 10: ss_trackball_l -> cs_user_l
- U2 pad 14: row5_l -> scl_l
- U2 pad 15: unconnected-(U2-Pad15) -> sda_l
- U2 pad 16: unconnected-(U2-Pad16) -> row3_l
- U2 pad 17: unconnected-(U2-Pad17) -> row5_l
- U2 pad 2: row2_l -> unconnected-(U2-Pad2)
- U2 pad 20: +3V3 -> unconnected-(U2-Pad20)
- U2 pad 26: split_hand_l -> button_user_l
- U2 pad 28: unconnected-(U2-Pad28) -> row2_l
- U2 pad 29: unconnected-(U2-Pad29) -> split_hand_l
- U2 pad 3: row3_l -> cs_trackball_l
- U2 pad 38: unconnected-(U2-Pad38) -> +3V3
- U2 pad 4: row4_l -> row1_l
- U2 pad 5: unconnected-(U2-Pad5) -> row4_l
- U2 pad 6: unconnected-(U2-Pad6) -> serial_l
Routing:
- net +5V: track 0.00 -> 60.9 mm
- net row1_l: track 0.00 -> 58.8 mm
- net cs_trackball_l: track 0.00 -> 56.3 mm, vias 0 -> 1
- net row4_l: track 0.00 -> 55.5 mm
- net col2_l: track 0.00 -> 53.6 mm
- net miso_l: track 0.00 -> 52.9 mm
- net col1_l: track 0.00 -> 51.9 mm
- net col3_l: track 0.00 -> 50.9 mm
- net mosi_l: track 0.00 -> 50.4 mm
- net sck_l: track 0.00 -> 48.9 mm, vias 0 -> 1
- net col4_l: track 0.00 -> 42.4 mm, vias 0 -> 1
- net col5_l: track 0.00 -> 42.1 mm, vias 0 -> 1
- net col6_l: track 0.00 -> 42.1 mm, vias 0 -> 1
- net row2_l: track 0.00 -> 38.6 mm, vias 0 -> 1
- net row5_l: track 0.00 -> 34.9 mm
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- removed copper zone on B.Cu, net Gnd2
- removed copper zone on F.Cu, net Gnd2
Other:
- board size 93.9 x 67.3 mm -> 93.8 x 67.7 mm
- board text added: "3V3"
- board text added: "5V"
- board text added: "Bastardkb x KarlK90"
- board text added: "CS"
- board text added: "Install Blackpill upside down together with ribbon cables and trs jack on this side. 5.1k resistors and push button on the opposite."
- board text added: "Install Blackpill, cables and jack on this side"
- board text added: "SCLK"
- board text added: "UPDATE"
- board text added: "VB"
- board text removed: "B0"
- board text removed: "D0"
- board text removed: "D1"
- board text removed: "Gnd"
- board text removed: "Install Elite-C, cables and jack on this side"
- board text removed: "REV 1.21"
- board text removed: "SCK"
- board text removed: "VCC"
- board text removed: "Vcc"

Commit message: silkscreen
Other:
- board text added: "BASTARDKB x KARLK90"
- board text removed: "Bastardkb x KarlK90"
Changed lines of the file:
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@@
     (pad "3" thru_hole oval locked (at 0 5.08) (size 1.7 1.7) (drill 1) (layers *.Cu *.Mask)
       (net 56 "rgb_l") (pinfunction "Pin_3") (pintype "passive"))
-    (model "${KICAD6_3DMODEL_DIR}/Connector_PinSocket_2.54mm.3dshapes/PinSocket_1x03_P2.54mm_Vertical.wrl"
+    (model "${KICAD6_3DMODEL_DIR}/Connector_PinSocket_2.54mm.3dshapes/PinSocket_1x03_P2.54mm_Vertical.wrl" hide
       (offset (xyz 0 0 0))
       (scale (xyz 1 1 1))
@@
     (pad "5" thru_hole oval locked (at 0 10.16) (size 1.7 1.7) (drill 1) (layers *.Cu *.Mask)
       (net 40 "row2_l") (pinfunction "Pin_5") (pintype "passive"))
-    (model "${KICAD6_3DMODEL_DIR}/Connector_PinHeader_2.54mm.3dshapes/PinHeader_1x05_P2.54mm_Vertical.wrl"
+    (model "${KICAD6_3DMODEL_DIR}/Connector_PinHeader_2.54mm.3dshapes/PinHeader_1x05_P2.54mm_Vertical.wrl" hide
       (offset (xyz 0 0 0))
       (scale (xyz 1 1 1))
@@
     )
   )
-  (gr_line (start 133.455 30.752112) (end 134.474111 30.752112) (layer "B.SilkS") (width 0.12))
-  (gr_arc (start 135.255 37.37319) (mid 135.024212 37.916441) (end 134.483922 38.154079) (layer "B.SilkS") (width 0.12))
-  (gr_arc (start 133.464811 38.154079) (mid 132.912917 37.914409) (end 132.683921 37.358001) (layer "B.SilkS") (width 0.12))
-  (gr_arc (start 134.474111 30.752112) (mid 135.026005 30.991782) (end 135.255001 31.54819) (layer "B.SilkS") (width 0.12))
-  (gr_line (start 132.683922 31.533001) (end 132.683921 37.358001) (layer "B.SilkS") (width 0.12))
-  (gr_arc (start 132.683922 31.533001) (mid 132.91471 30.98975) (end 133.455 30.752112) (layer "B.SilkS") (width 0.12))
-  (gr_line (start 135.255 37.37319) (end 135.255 31.54819) (layer "B.SilkS") (width 0.12))
-  (gr_line (start 134.483922 38.154079) (end 133.464811 38.154079) (layer "B.SilkS") (width 0.12))
+  (gr_line (start 131.171079 29.094111) (end 132.19019 29.094111) (layer "B.SilkS") (width 0.12))
+  (gr_arc (start 132.971079 35.715189) (mid 132.740291 36.25844) (end 132.200001 36.496078) (layer "B.SilkS") (width 0.12))
+  (gr_arc (start 131.18089 36.496078) (mid 130.628996 36.256408) (end 130.4 35.7) (layer "B.SilkS") (width 0.12))
+  (gr_arc (start 132.19019 29.094111) (mid 132.742084 29.333781) (end 132.97108 29.890189) (layer "B.SilkS") (width 0.12))
+  (gr_line (start 130.400001 29.875) (end 130.4 35.7) (layer "B.SilkS") (width 0.12))
+  (gr_arc (start 130.400001 29.875) (mid 130.630789 29.331749) (end 131.171079 29.094111) (layer "B.SilkS") (width 0.12))
+  (gr_line (start 132.971079 35.715189) (end 132.971079 29.890189) (layer "B.SilkS") (width 0.12))
+  (gr_line (start 132.200001 36.496078) (end 131.18089 36.496078) (layer "B.SilkS") (width 0.12))
   (gr_line (start 116.327011 36.135878) (end 115.3079 36.135878) (layer "F.SilkS") (width 0.12))
-  (gr_arc (start 133.455 38.154079) (mid 132.91471 37.916441) (end 132.683922 37.37319) (layer "F.SilkS") (width 0.12))
-  (gr_line (start 132.683922 31.54819) (end 132.683922 37.37319) (layer "F.SilkS") (width 0.12))
-  (gr_arc (start 134.483922 30.752112) (mid 135.024212 30.98975) (end 135.255 31.533001) (layer "F.SilkS") (width 0.12))
+  (gr_arc (start 131.171079 36.496078) (mid 130.630789 36.25844) (end 130.400001 35.715189) (layer "F.SilkS") (width 0.12))
+  (gr_line (start 130.400001 29.890189) (end 130.400001 35.715189) (layer "F.SilkS") (width 0.12))
+  (gr_arc (start 132.200001 29.094111) (mid 132.740291 29.331749) (end 132.971079 29.875) (layer "F.SilkS") (width 0.12))
   (gr_arc (start 117.107901 35.3398) (mid 116.878905 35.896208) (end 116.327011 36.135878) (layer "F.SilkS") (width 0.12))
   (gr_rect (start 90.351 32.28) (end 82.241 16.28) (layer "F.SilkS") (width 0.15) (fill none))
   (gr_arc (start 116.336822 28.733911) (mid 116.877112 28.971549) (end 117.1079 29.5148) (layer "F.SilkS") (width 0.12))
   (gr_rect (start 165.811 32.18) (end 157.701 16.18) (layer "F.SilkS") (width 0.15) (fill none))
-  (gr_line (start 133.464811 30.752112) (end 134.483922 30.752112) (layer "F.SilkS") (width 0.12))
-  (gr_arc (start 135.255001 37.358001) (mid 135.026005 37.914409) (end 134.474111 38.154079) (layer "F.SilkS") (width 0.12))
-  (gr_line (start 134.474111 38.154079) (end 133.455 38.154079) (layer "F.SilkS") (width 0.12))
-  (gr_arc (start 132.683921 31.54819) (mid 132.912917 30.991782) (end 133.464811 30.752112) (layer "F.SilkS") (width 0.12))
+  (gr_line (start 131.18089 29.094111) (end 132.200001 29.094111) (layer "F.SilkS") (width 0.12))
+  (gr_arc (start 132.97108 35.7) (mid 132.742084 36.256408) (end 132.19019 36.496078) (layer "F.SilkS") (width 0.12))
+  (gr_line (start 132.19019 36.496078) (end 131.171079 36.496078) (layer "F.SilkS") (width 0.12))
+  (gr_arc (start 130.4 29.890189) (mid 130.628996 29.333781) (end 131.18089 29.094111) (layer "F.SilkS") (width 0.12))
   (gr_line (start 115.317711 28.733911) (end 116.336822 28.733911) (layer "F.SilkS") (width 0.12))
   (gr_arc (start 114.536821 29.529989) (mid 114.765817 28.973581) (end 115.317711 28.733911) (layer "F.SilkS") (width 0.12))
   (gr_line (start 117.107901 35.3398) (end 117.1079 29.5148) (layer "F.SilkS") (width 0.12))
-  (gr_line (start 135.255001 37.358001) (end 135.255 31.533001) (layer "F.SilkS") (width 0.12))
+  (gr_line (start 132.97108 35.7) (end 132.971079 29.875) (layer "F.SilkS") (width 0.12))
   (gr_arc (start 115.3079 36.135878) (mid 114.76761 35.89824) (end 114.536822 35.354989) (layer "F.SilkS") (width 0.12))
   (gr_line (start 114.536822 29.529989) (end 114.536822 35.354989) (layer "F.SilkS") (width 0.12))
@@
   (gr_arc (start 155.94 21.34) (mid 155.247256 21.665951) (end 154.487106 21.757106) (layer "Edge.Cuts") (width 0.2))
   (gr_line (start 112.686922 46.157609) (end 119.166648 33.968362) (layer "Edge.Cuts") (width 0.2))
-  (gr_arc (start 164.88 20.93) (mid 165.913543 21.36974) (end 166.341679 22.408144) (layer "Edge.Cuts") (width 0.2))
+  (gr_arc (start 164.88 20.93) (mid 165.913544 21.36974) (end 166.341679 22.408144) (layer "Edge.Cuts") (width 0.2))
   (gr_line (start 129.800867 35.6) (end 134.3 44) (layer "Edge.Cuts") (width 0.2))
   (gr_line (start 119.423514 25.217534) (end 119.339931 32.952692) (layer "Edge.Cuts") (width 0.2))
@@
     (effects (font (size 0.8 0.8) (thickness 0.15)) (justify mirror))
   )
-  (gr_text "BLACKPILL HOLDER 0.1" (at 136.8044 60.8076 -90) (layer "B.SilkS")
-    (effects (font (size 1.016 1.016) (thickness 0.1524)) (justify mirror))
+  (gr_text "BLACKPILL HOLDER 0.1" (at 134.5 34.992858 -90) (layer "B.SilkS")
+    (effects (font (size 0.8 0.8) (thickness 0.15)) (justify mirror))
   )
   (gr_text "UPDATE" (at 147.193 70.3072) (layer "B.SilkS")
@@
     (effects (font (size 0.8 0.8) (thickness 0.15)) (justify mirror))
   )
-  (gr_text "Bastardkb x KarlK90" (at 157.5308 61.6966 270) (layer "B.SilkS")
-    (effects (font (size 1.016 1.016) (thickness 0.1524)) (justify mirror))
+  (gr_text "BASTARDKB x KARLK90" (at 135.95 35.05 270) (layer "B.SilkS")
+    (effects (font (size 0.8 0.8) (thickness 0.15)) (justify mirror))
   )
   (gr_text "MOSI" (at 96.881864 78.5622) (layer "B.SilkS")
@@
     (effects (font (size 0.8 0.8) (thickness 0.15)) (justify mirror))
   )
-  (gr_text "LEFT" (at 133.883921 34.233001 -90) (layer "B.SilkS")
+  (gr_text "LEFT" (at 131.6 32.575 -90) (layer "B.SilkS")
     (effects (font (size 1.5 1.5) (thickness 0.2)) (justify mirror))
   )
@@
     (effects (font (size 1.2 1.2) (thickness 0.15)))
   )
-  (gr_text "LEFT" (at 134.055001 34.233001 90) (layer "F.SilkS")
+  (gr_text "LEFT" (at 131.77108 32.575 90) (layer "F.SilkS")
     (effects (font (size 1.5 1.5) (thickness 0.2)))
   )
@@
     (effects (font (size 0.8 0.8) (thickness 0.15)))
   )
+  (gr_text "GITHUB.COM/BASTARDKB" (at 134.55 34.75 90) (layer "F.SilkS")
+    (effects (font (size 0.8 0.8) (thickness 0.15)))
+  )
   (gr_text "R2" (at 146.688177 83.6422) (layer "F.SilkS")
     (effects (font (size 0.8 0.8) (thickness 0.15)))
@@
   )
   (gr_text "Install Blackpill\nupside down\ntogether with \nribbon cables\nand trs jack\non this side.\n\n5.1k resistors\nand push button\non the opposite." (at 147.2 55.58) (layer "F.SilkS")
-    (effects (font (size 0.9652 0.9652) (thickness 0.14732)))
+    (effects (font (size 0.8 0.8) (thickness 0.15)))
+  )
+  (gr_text "BASTARDKB.COM" (at 136.1 37.302381 90) (layer "F.SilkS")
+    (effects (font (size 0.8 0.8) (thickness 0.15)))
   )
   (gr_text "todo\n- version number\n- check onboard buttons are accessible\n- check edge cuts\n- change board name" (at 179.25 32.7) (layer "F.Fab")
@@
     )
   )
+  (group "" (id 399191b8-8b7b-4250-8232-13bcd8d54727)
+    (members
+      755dcd2b-1a0d-4674-94fa-28c95292f593
+      ef9ac040-5faf-488d-b7bc-ebf588cbf6e1
+    )
+  )
   (group "" (id 4817069f-538a-428b-bb7d-d2f633c6eeae)
     (members
@@
     )
   )
-  (group "" (id e3e88b48-77ab-45bd-9335-8076eb260601)
-    (members
-      755dcd2b-1a0d-4674-94fa-28c95292f593
-      ef9ac040-5faf-488d-b7bc-ebf588cbf6e1
-    )
-  )

Commit message: edge cuts
Parts:
- moved G*** 3.73 mm to (124.0, 62.0), turned to 90 degrees
- moved G*** 3.56 mm to (124.0, 61.9), turned to -90 degrees
Other:
- board size 93.8 x 67.7 mm -> 93.5 x 67.4 mm
