File: adapter/adapter.kicad_pcb (KiCad board)
At the start: 2 copper layers, 93.5 x 67.4 mm, 32 parts, among them J1 Serial, J10 Ribbon, J11 SPI user, J12 SPI user, J2 Serial, J3 RGB, J4 RGB, J5 Trackball, J6 Ribbon, J7 Trackball, J8 Ribbon, J9 Ribbon, SW1 USER, SW2 USER, U1 STM32F401 / STM32F411 Blackpi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, U2 STM32F401 / STM32F411 Blackpi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

Commit message: silkscreen
Other:
- board text added: "2021 QUENTIN LEBASTARD BASTARD KEYBOARDS"
- board text removed: "2021 QUENTIN LEBASTARD"
- board text removed: "CHARYBDIS HOLDER"
- board text removed: "Have a fun build"

Commit message: add license
Other:
- board text added: "Licensed under CERN-OHL-W v2"
Changed lines of the file:
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@@
     (effects (font (size 0.8 0.8) (thickness 0.15)) (justify mirror))
+  )
+  (gr_text "Licensed under \nCERN-OHL-W v2" (at 124.6 84) (layer "B.SilkS")
+    (effects (font (size 0.8 0.8) (thickness 0.12)) (justify mirror))
   )
   (gr_text "GND" (at 152.75 86.18) (layer "B.SilkS")
@@
     (effects (font (size 0.8 0.8) (thickness 0.15)))
   )
+  (gr_text "Licensed under \nCERN-OHL-W v2" (at 124.85 83.9) (layer "F.SilkS")
+    (effects (font (size 0.8 0.8) (thickness 0.12)))
+  )
   (gr_text "R5" (at 111.3028 86.1822) (layer "F.SilkS")

Commit message: silkscreen
Parts:
- moved J6 2.74 mm to (98.4, 73.5)
- moved J8 1.00 mm to (109.8, 73.5)
- moved J7 0.80 mm to (92.7, 73.5)
- moved J12 0.73 mm to (104.1, 73.5)
Other:
- board text removed: "SC"
- board text removed: "SS"
