File: adapter/adapter.kicad_pcb (KiCad board)
At the start: 2 copper layers, 93.5 x 67.4 mm, 32 parts, among them J1 Serial, J10 Ribbon, J11 SPI user, J12 SPI user, J2 Serial, J3 RGB, J4 RGB, J5 Trackball, J6 Ribbon, J7 Trackball, J8 Ribbon, J9 Ribbon, SW1 USER, SW2 USER, U1 STM32F401 / STM32F411 Blackpi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, U2 STM32F401 / STM32F411 Blackpi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

Commit message: Release Candidate
Parts:
- moved R7 8.15 mm to (101.2, 42.3), turned to 90 degrees
- moved R6 7.27 mm to (105.2, 42.3), turned to 90 degrees
- moved J12 5.66 mm to (98.4, 73.5)
- moved J6 5.61 mm to (104.0, 73.5)
- moved R8 3.08 mm to (97.2, 42.3), turned to 90 degrees
- moved J8 0.16 mm to (109.6, 73.5)
- moved J7 0.12 mm to (92.9, 73.5)
Connections:
- U1 pad 10: cs_user_l -> cs_user_r
- U1 pad 20: unconnected-(U1-Pad20) -> +3V3
- U1 pad 30: unconnected-(U1-Pad30) -> cs_eeprom_r
- U1 pad 38: +3V3 -> unconnected-(U1-Pad38)
- U1 pad 6: unconnected-(U1-Pad6) -> serial_r
- U2 pad 30: unconnected-(U2-Pad30) -> cs_eeprom_l
Routing:
- net col3_r: track 0.00 -> 77.4 mm
- net +5V: track 60.9 -> 131.7 mm
- net mosi_r: track 0.00 -> 64.3 mm
- net cs_trackball_r: track 0.00 -> 61.0 mm
- net col1_r: track 0.00 -> 53.6 mm
- net col2_r: track 0.00 -> 52.7 mm
- net row1_r: track 0.00 -> 51.9 mm, vias 0 -> 1
- net miso_r: track 0.00 -> 50.3 mm
- net serial_r: track 0.00 -> 49.2 mm, vias 0 -> 2
- net row4_r: track 0.00 -> 48.9 mm
- net sck_r: track 0.00 -> 44.9 mm
- net row2_r: track 0.00 -> 40.5 mm
- net cs_user_r: track 0.00 -> 38.5 mm, vias 0 -> 1
- net col4_r: track 0.00 -> 37.2 mm
- net col5_r: track 0.00 -> 36.5 mm
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Other:
- board text added: "2021 QUENTIN LEBASTARD AND STEFAN KERKMANN"
- board text added: "MATRIX"
- board text added: "SCL"
- board text added: "SDA"
- board text added: "SPI"
- board text removed: "2021 QUENTIN LEBASTARD BASTARD KEYBOARDS"
- board text removed: "Install Blackpill, cables and jack on this side"
- board text removed: "todo - version number - check onboard buttons are accessible - check edge cuts - change board name"

Commit message: silkscren around serial
Other:
- board text added: "BLACKPILL HOLDER 1.0"
- board text removed: "BLACKPILL HOLDER 0.1"
Changed lines of the file:
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@@
   (gr_arc (start 116.861194 29.137703) (mid 117.413088 29.377373) (end 117.642084 29.933781) (layer "B.SilkS") (width 0.12))
   (gr_line (start 115.842083 29.137703) (end 116.861194 29.137703) (layer "B.SilkS") (width 0.12))
+  (gr_rect (start 158.09 32.35) (end 165.48 20.29) (layer "B.SilkS") (width 0.15) (fill none))
+  (gr_rect (start 82.675 32.21) (end 90.065 20.15) (layer "B.SilkS") (width 0.15) (fill none))
   (gr_line (start 132.971079 35.715189) (end 132.971079 29.890189) (layer "B.SilkS") (width 0.12))
   (gr_arc (start 117.642083 35.758781) (mid 117.411295 36.302032) (end 116.871005 36.53967) (layer "B.SilkS") (width 0.12))
@@
   (gr_arc (start 116.979307 29.148192) (mid 117.519597 29.38583) (end 117.750385 29.929081) (layer "F.SilkS") (width 0.12))
   (gr_line (start 131.18089 29.094111) (end 132.200001 29.094111) (layer "F.SilkS") (width 0.12))
+  (gr_rect (start 82.72 20.18) (end 90.11 32.24) (layer "F.SilkS") (width 0.15) (fill none))
   (gr_arc (start 132.97108 35.7) (mid 132.742084 36.256408) (end 132.19019 36.496078) (layer "F.SilkS") (width 0.12))
+  (gr_rect (start 158.135 20.32) (end 165.525 32.38) (layer "F.SilkS") (width 0.15) (fill none))
   (gr_line (start 132.19019 36.496078) (end 131.171079 36.496078) (layer "F.SilkS") (width 0.12))
   (gr_arc (start 130.4 29.890189) (mid 130.628996 29.333781) (end 131.18089 29.094111) (layer "F.SilkS") (width 0.12))
@@
   (gr_arc (start 168.66 49.42) (mid 170.815116 54.143025) (end 166.718015 57.331325) (layer "Edge.Cuts") (width 0.2))
   (gr_line (start 91.049999 20.873353) (end 83.499999 20.876401) (layer "Edge.Cuts") (width 0.2))
-  (gr_arc (start 115.191776 76.100339) (mid 114.539171 77.119389) (end 113.339996 76.957105) (layer "Edge.Cuts") (width 0.2))
+  (gr_arc (start 115.191776 76.100339) (mid 114.539171 77.119387) (end 113.339997 76.957104) (layer "Edge.Cuts") (width 0.2))
   (gr_line (start 153.487106 22.757106) (end 153.490247 37.692893) (layer "Edge.Cuts") (width 0.2))
   (gr_circle (center 112.938071 54.271409) (end 112.938071 53.871409) (layer "Edge.Cuts") (width 0.2) (fill none))
@@
     (effects (font (size 0.8 0.8) (thickness 0.15)) (justify mirror))
   )
-  (gr_text "BLACKPILL HOLDER 0.1" (at 112.15 35.690477 -90) (layer "B.SilkS")
+  (gr_text "BLACKPILL HOLDER 1.0" (at 112.15 35.690477 -90) (layer "B.SilkS")
     (effects (font (size 0.8 0.8) (thickness 0.15)) (justify mirror))
   )
@@
     (effects (font (size 0.8 0.8) (thickness 0.15)) (justify mirror))
   )
-  (gr_text "BLACKPILL HOLDER 0.1" (at 134.5 35.690477 -90) (layer "B.SilkS")
-    (effects (font (size 0.8 0.8) (thickness 0.15)) (justify mirror))
-  )
+  (gr_text "BLACKPILL HOLDER 1.0" (at 134.5 35.690477 -90) (layer "B.SilkS")
+    (effects (font (size 0.8 0.8) (thickness 0.15)) (justify mirror))
+  )

Commit message: Bugfix release 1.1
PB2 has a pulldown on the WeACT board to ensure BOOT1
is low during boot up. Otherwise jumping into the bootloader
is not ensured. So COL3 is moved from PB2 to PB10 as the pull
down prevents this pin from beeing used for matrix scanning.
Parts:
- turned G*** to 90 degrees
Connections:
- U1 pad 36: col3_r -> unconnected-(U1-Pad36)
- U1 pad 37: unconnected-(U1-Pad37) -> col3_r
- U2 pad 36: col3_l -> unconnected-(U2-Pad36)
- U2 pad 37: unconnected-(U2-Pad37) -> col3_l
Routing:
- net col3_l: track 51.2 -> 53.8 mm
- net col3_r: track 77.4 -> 79.9 mm
Other:
- board text added: "BLACKPILL HOLDER 1.1"
- board text removed: "BLACKPILL HOLDER 1.0"
Changed lines of the file:
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@@
     (title "Bastardkb Blackpill Holder")
     (date "2021-12-08")
-    (rev "0.1")
+    (rev "1.1")
   )
   (layers
@@
       (usegerberattributes true)
       (usegerberadvancedattributes true)
-      (creategerberjobfile true)
+      (creategerberjobfile false)
       (svguseinch false)
       (svgprecision 6)
@@
       (viasonmask false)
       (mode 1)
-      (useauxorigin true)
+      (useauxorigin false)
       (hpglpennumber 1)
       (hpglpenspeed 20)
@@
   (net 16 "row2_r")
   (net 17 "row3_r")
-  (net 18 "unconnected-(U1-Pad37)")
+  (net 18 "unconnected-(U1-Pad36)")
   (net 19 "row4_r")
   (net 20 "col3_r")
@@
   (net 40 "row2_l")
   (net 41 "row3_l")
-  (net 42 "unconnected-(U2-Pad37)")
+  (net 42 "unconnected-(U2-Pad36)")
   (net 43 "row4_l")
   (net 44 "col3_l")
@@
       (net 45 "col2_l") (pinfunction "PB1") (pintype "bidirectional"))
     (pad "36" thru_hole circle locked (at 15.24 -10.16 180) (size 1.7 1.7) (drill 1) (layers *.Cu *.Mask)
-      (net 44 "col3_l") (pinfunction "PB2") (pintype "bidirectional"))
+      (net 42 "unconnected-(U2-Pad36)") (pinfunction "PB2") (pintype "bidirectional+no_connect"))
     (pad "37" thru_hole circle locked (at 15.24 -7.62 180) (size 1.7 1.7) (drill 1) (layers *.Cu *.Mask)
-      (net 42 "unconnected-(U2-Pad37)") (pinfunction "PB10") (pintype "bidirectional+no_connect"))
+      (net 44 "col3_l") (pinfunction "PB10") (pintype "bidirectional"))
     (pad "38" thru_hole circle locked (at 15.24 -5.08 180) (size 1.7 1.7) (drill 1) (layers *.Cu *.Mask)
       (net 38 "+3V3") (pinfunction "3V3") (pintype "power_in"))
@@
   )
   (footprint "LOGO" (layer "B.Cu")
-    (at 124 61.9 -90)
+    (at 124 61.9 90)
     (attr board_only exclude_from_pos_files exclude_from_bom)
-    (fp_text reference "G***" (at 0 0 -270) (layer "B.SilkS") hide
+    (fp_text reference "G***" (at 0 0 90) (layer "B.SilkS") hide
       (effects (font (size 1.524 1.524) (thickness 0.3)) (justify mirror))
     )
-    (fp_text value "LOGO" (at 0.75 0 -270) (layer "B.SilkS") hide
+    (fp_text value "LOGO" (at 0.75 0 90) (layer "B.SilkS") hide
       (effects (font (size 1.524 1.524) (thickness 0.3)) (justify mirror))
     )
@@
       (net 22 "col2_r") (pinfunction "PB1") (pintype "bidirectional"))
     (pad "36" thru_hole circle locked (at 15.24 -10.16 180) (size 1.7 1.7) (drill 1) (layers *.Cu *.Mask)
-      (net 20 "col3_r") (pinfunction "PB2") (pintype "bidirectional"))
+      (net 18 "unconnected-(U1-Pad36)") (pinfunction "PB2") (pintype "bidirectional+no_connect"))
     (pad "37" thru_hole circle locked (at 15.24 -7.62 180) (size 1.7 1.7) (drill 1) (layers *.Cu *.Mask)
-      (net 18 "unconnected-(U1-Pad37)") (pinfunction "PB10") (pintype "bidirectional+no_connect"))
+      (net 20 "col3_r") (pinfunction "PB10") (pintype "bidirectional"))
     (pad "38" thru_hole circle locked (at 15.24 -5.08 180) (size 1.7 1.7) (drill 1) (layers *.Cu *.Mask)
       (net 23 "unconnected-(U1-Pad38)") (pinfunction "3V3") (pintype "power_in+no_connect"))
@@
     (effects (font (size 0.8 0.8) (thickness 0.15)) (justify mirror))
   )
-  (gr_text "BLACKPILL HOLDER 1.0" (at 112.15 35.690477 -90) (layer "B.SilkS")
+  (gr_text "BLACKPILL HOLDER 1.1" (at 112.15 35.690477 -90) (layer "B.SilkS")
     (effects (font (size 0.8 0.8) (thickness 0.15)) (justify mirror))
   )
@@
     (effects (font (size 0.8 0.8) (thickness 0.15)) (justify mirror))
   )
-  (gr_text "BLACKPILL HOLDER 1.0" (at 134.5 35.690477 -90) (layer "B.SilkS")
+  (gr_text "BLACKPILL HOLDER 1.1" (at 134.5 35.690477 -90) (layer "B.SilkS")
     (effects (font (size 0.8 0.8) (thickness 0.15)) (justify mirror))
   )
@@
   (segment (start 109.619999 73.4822) (end 110.584711 72.517488) (width 0.2032) (layer "B.Cu") (net 19))
   (segment (start 110.255 43.979) (end 110.255 32.041) (width 0.2032) (layer "B.Cu") (net 19))
-  (segment (start 100.857 55.536) (end 97.555 52.234) (width 0.2032) (layer "B.Cu") (net 20))
-  (segment (start 104.031998 73.4822) (end 105.556 75.006202) (width 0.2032) (layer "B.Cu") (net 20))
-  (segment (start 105.556 75.006202) (end 105.556 83.984) (width 0.2032) (layer "B.Cu") (net 20))
-  (segment (start 92.670282 52.234) (end 91.561578 51.125296) (width 0.2032) (layer "B.Cu") (net 20))
-  (segment (start 91.561578 32.688422) (end 93.54 30.71) (width 0.2032) (layer "B.Cu") (net 20))
-  (segment (start 97.555 52.234) (end 92.670282 52.234) (width 0.2032) (layer "B.Cu") (net 20))
-  (segment (start 91.561578 51.125296) (end 91.561578 32.688422) (width 0.2032) (layer "B.Cu") (net 20))
-  (segment (start 100.857 83.984) (end 100.857 55.536) (width 0.2032) (layer "B.Cu") (net 20))
-  (segment (start 104.667 84.873) (end 101.746 84.873) (width 0.2032) (layer "B.Cu") (net 20))
-  (segment (start 105.556 83.984) (end 104.667 84.873) (width 0.2032) (layer "B.Cu") (net 20))
-  (segment (start 101.746 84.873) (end 100.857 83.984) (width 0.2032) (layer "B.Cu") (net 20))
+  (segment (start 92.670282 52.234) (end 97.555 52.234) (width 0.2032) (layer "B.Cu") (net 20))
+  (segment (start 91.561578 30.148422) (end 91.561578 51.125296) (width 0.2032) (layer "B.Cu") (net 20))
+  (segment (start 105.556 83.984) (end 105.556 75.006202) (width 0.2032) (layer "B.Cu") (net 20))
+  (segment (start 93.54 28.17) (end 91.561578 30.148422) (width 0.2032) (layer "B.Cu") (net 20))
+  (segment (start 100.857 55.536) (end 100.857 83.984) (width 0.2032) (layer "B.Cu") (net 20))
+  (segment (start 104.667 84.873) (end 105.556 83.984) (width 0.2032) (layer "B.Cu") (net 20))
+  (segment (start 100.857 83.984) (end 101.746 84.873) (width 0.2032) (layer "B.Cu") (net 20))
+  (segment (start 91.561578 51.125296) (end 92.670282 52.234) (width 0.2032) (layer "B.Cu") (net 20))
+  (segment (start 101.746 84.873) (end 104.667 84.873) (width 0.2032) (layer "B.Cu") (net 20))
+  (segment (start 105.556 75.006202) (end 104.031998 73.4822) (width 0.2032) (layer "B.Cu") (net 20))
+  (segment (start 97.555 52.234) (end 100.857 55.536) (width 0.2032) (layer "B.Cu") (net 20))
   (segment (start 110.255 70.649) (end 110.255 62.648) (width 0.2032) (layer "B.Cu") (net 21))
   (segment (start 109.619999 86.1822) (end 108.096 84.658201) (width 0.2032) (layer "B.Cu") (net 21))
@@
   (segment (start 139.042954 73.4822) (end 142.894 69.631154) (width 0.2032) (layer "B.Cu") (net 43))
   (segment (start 142.894 69.631154) (end 142.894 66.911848) (width 0.2032) (layer "B.Cu") (net 43))
-  (segment (start 137.414 50.945) (end 137.414 32.9184) (width 0.2032) (layer "F.Cu") (net 44))
-  (segment (start 143.8402 52.2732) (end 138.7422 52.2732) (width 0.2032) (layer "F.Cu") (net 44))
-  (segment (start 146.323 54.756) (end 143.8402 52.2732) (width 0.2032) (layer "F.Cu") (net 44))
-  (segment (start 146.323 71.609) (end 146.323 54.756) (width 0.2032) (layer "F.Cu") (net 44))
-  (segment (start 137.414 32.9184) (end 139.6238 30.7086) (width 0.2032) (layer "F.Cu") (net 44))
-  (segment (start 144.399 73.533) (end 146.323 71.609) (width 0.2032) (layer "F.Cu") (net 44))
-  (segment (start 138.7422 52.2732) (end 137.414 50.945) (width 0.2032) (layer "F.Cu") (net 44))
+  (segment (start 146.323 71.609) (end 144.399 73.533) (width 0.2032) (layer "F.Cu") (net 44))
+  (segment (start 143.8402 52.2732) (end 146.323 54.756) (width 0.2032) (layer "F.Cu") (net 44))
+  (segment (start 137.414 30.366) (end 137.414 50.945) (width 0.2032) (layer "F.Cu") (net 44))
+  (segment (start 139.62 28.16) (end 137.414 30.366) (width 0.2032) (layer "F.Cu") (net 44))
+  (segment (start 137.414 50.945) (end 138.7422 52.2732) (width 0.2032) (layer "F.Cu") (net 44))
+  (segment (start 138.7422 52.2732) (end 143.8402 52.2732) (width 0.2032) (layer "F.Cu") (net 44))
+  (segment (start 146.323 54.756) (end 146.323 71.609) (width 0.2032) (layer "F.Cu") (net 44))
   (segment (start 147.014701 76.759299) (end 147.014701 54.431701) (width 0.2032) (layer "F.Cu") (net 45))
   (segment (start 147.014701 54.431701) (end 142.367 49.784) (width 0.2032) (layer "F.Cu") (net 45))

Commit message: Start rev1.2 and move update button 3.75mm up
Parts:
- moved SW1 3.75 mm to (147.2, 61.1)
- moved SW2 3.75 mm to (101.2, 61.1)
- moved G*** 1.10 mm to (147.3, 50.9)
- moved G*** 1.10 mm to (101.2, 50.9)
Routing:
- net row1_l: track 58.8 -> 61.0 mm
- net row5_l: track 34.3 -> 36.5 mm
- net button_user_r: track 14.3 -> 12.9 mm
- net row3_l: track 26.8 -> 28.2 mm
- net row4_l: track 54.1 -> 55.1 mm
- net col6_l: track 42.0 -> 42.9 mm
- net button_user_l: track 14.1 -> 13.2 mm
- net col5_l: track 42.1 -> 43.0 mm
- net col4_l: track 41.9 -> 42.8 mm
- net GND: vias 29 -> 28
Other:
- board text added: "2022 QUENTIN LEBASTARD AND STEFAN KERKMANN"
- board text added: "BLACKPILL HOLDER 1.2"
- board text removed: "2021 QUENTIN LEBASTARD AND STEFAN KERKMANN"
- board text removed: "BLACKPILL HOLDER 1.1"

Commit message: change edge cuts to have more space for ribbon cables
Other:
- outline, holes or cut-outs redrawn
- board text removed: "BASTARDKB.COM"

Commit message: Add I2C header to schematic, start placement
Parts:
- added J13: I2C, Library:4_PinHeader, F.Cu at (160.5, 78.1)
- added J14: I2C, Library:4_PinHeader, F.Cu at (87.5, 78.6)
- added R10: 5.1k, Resistor_SMD:R_1206_3216Metric_Pad1.30x1.75mm_HandSolder, F.Cu at (159.0, 54.6)
- added R11: 5.1k, Resistor_SMD:R_1206_3216Metric_Pad1.30x1.75mm_HandSolder, F.Cu at (159.0, 49.6)
- added R12: 5.1k, Resistor_SMD:R_1206_3216Metric_Pad1.30x1.75mm_HandSolder, F.Cu at (90.0, 53.6)
- added R9: 5.1k, Resistor_SMD:R_1206_3216Metric_Pad1.30x1.75mm_HandSolder, F.Cu at (87.5, 53.6)
Routing:
- net serial_r: track 49.2 -> 78.7 mm, vias 2 -> 3
- net cs_trackball_r: track 61.0 -> 45.4 mm
- net dfu_bootloader_bodge_r: track 13.9 -> 0.00 mm, vias 1 -> 0
Other:
- board text removed: "SCL"
- board text removed: "SDA"
